File: electronics/RovHat/RovHat.kicad_pcb (KiCad board)
At the start: 4 copper layers, 85 x 56 mm, 47 parts, among them J201 ADS1115, J202 ANALOG INPUT, J203 GYRO, J301 PWM_OUT, J305 SWD_EXT, J401 RPI Header, J402 USB_A, J403 DEPTH, J404 PROPULSION, J501 OUT1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

Commit message: Final Version
Parts:
- removed J506: PWR IN, Connector_Phoenix_MC:PhoenixContact_MCV_1,5_2-G-3.5_1x02_P3.50mm_Vertical
- removed J507: PWR OUT, Connector_PinHeader_2.54mm:PinHeader_1x02_P2.54mm_Vertical
- removed J508: PWR OUT2, Connector_Phoenix_MC:PhoenixContact_MCV_1,5_2-G-3.5_1x02_P3.50mm_Vertical
- added J204: I2C EXPAND, Connector_PinHeader_2.54mm:PinHeader_1x04_P2.54mm_Vertical, F.Cu at (145.5, 127.1)
- added R401: 0R, Resistor_SMD:R_0603_1608Metric, F.Cu at (144.2, 139.3)
- added R402: 0R, Resistor_SMD:R_0603_1608Metric, F.Cu at (141.6, 139.3)
- J501, J502: footprint Connector_Phoenix_MC:PhoenixContact_MCV_1,5_2-G-3.5_1x02_P3.50mm_Vertical -> Connector_Phoenix_MC:PhoenixContact_MCV_1,5_4-G-3.5_1x04_P3.50mm_Vertical
- J503: value OUT3 -> PWR; footprint Connector_Phoenix_MC:PhoenixContact_MCV_1,5_2-G-3.5_1x02_P3.50mm_Vertical -> Connector_Phoenix_MC:PhoenixContact_MCV_1,5_4-G-3.5_1x04_P3.50mm_Vertical
- J505: value OUT4 -> PWR_IN; footprint Connector_Phoenix_MC:PhoenixContact_MCV_1,5_2-G-3.5_1x02_P3.50mm_Vertical -> Connector_PinHeader_2.54mm:PinHeader_2x02_P2.54mm_Vertical
- moved J504 62.0 mm to (88.9, 109.7), turned to 90 degrees
- moved J503 33.3 mm to (98.6, 97.3), turned to 0 degrees
- moved J505 11.1 mm to (147.7, 103.0), turned to 90 degrees
- moved J502 9.22 mm to (131.9, 97.3), turned to 0 degrees
- moved J501 2.85 mm to (115.3, 97.3), turned to 0 degrees
Connections:
- J401 pad 2: +5V -> Net-(J401-Pad2)
- J401 pad 4: +5V -> Net-(J401-Pad2)
- J502 pad 2: Net-(D502-Pad1) -> Net-(D503-Pad1)
- J503 pad 2: Net-(D503-Pad1) -> GND
- J505 pad 2: Net-(D504-Pad1) -> +VSW
Routing:
- net /MCU/GYRO_INT: track 30.9 -> 33.6 mm
- net VDD: track 69.6 -> 72.2 mm
- net /Sensors/SDA: track 84.1 -> 85.7 mm
- net /Sensors/SCL: track 72.8 -> 74.3 mm
- net /Connectors/RPI_RXD: track 32.9 -> 32.4 mm
- net +5V: vias 2 -> 9
- added copper zone on F.Cu, net +5V
- added copper zone on F.Cu, net Net-(J401-Pad2)
