File: electronics/RovHat/RovHat.kicad_pcb (KiCad board)
At the start: 4 copper layers, 85 x 56 mm, 47 parts, among them J201 ADS1115, J202 ANALOG INPUT, J203 GYRO, J204 I2C EXPAND, J301 PWM_OUT, J305 SWD_EXT, J401 RPI Header, J402 USB_A, J403 DEPTH, J404 PROPULSION, J501 OUT1, J502 OUT2, J503 PWR, J504 5V IN, J505 PWR_IN, Q501 IRF7403, Q502 IRF7403, Q503 IRF7403, Q504 IRF7403, U301 Rpi_Pico

Commit message: Multiple fixes
Parts:
- removed D501, D502: MBR0550, Diode_SMD:D_SOD-123
- removed J201: ADS1115, Connector_PinHeader_2.54mm:PinHeader_1x10_P2.54mm_Vertical
- removed J402: USB_A, Connector_USB:USB_A_Molex_67643_Horizontal
- removed J404: PROPULSION, Connector_PinHeader_2.54mm:PinHeader_1x06_P2.54mm_Vertical
- removed J501: OUT1, Connector_Phoenix_MC:PhoenixContact_MCV_1,5_4-G-3.5_1x04_P3.50mm_Vertical
- removed Q501, Q502: IRF7403, Package_SO:SOIC-8_3.9x4.9mm_P1.27mm
- removed R501, R502: R_Small, Resistor_SMD:R_0603_1608Metric
- removed REF**: Logo, Findersee_parts:Logo
- added C1: 1uf, Capacitor_SMD:C_0603_1608Metric, F.Cu at (69.7, 141.9)
- added C2: 2u2, Capacitor_SMD:C_0805_2012Metric, F.Cu at (124.5, 105.9)
- added C3: 2u2, Capacitor_SMD:C_0805_2012Metric, F.Cu at (124.5, 108.0)
- added F1: Polyfuse, Fuse:Fuse_1206_3216Metric, B.Cu at (133.4, 93.8)
- added F2: Polyfuse, Fuse:Fuse_1206_3216Metric, F.Cu at (100.0, 102.2)
- added F3: Polyfuse, Fuse:Fuse_1206_3216Metric, B.Cu at (140.4, 93.8)
- added J11: Depth, Connector_PinHeader_2.54mm:PinHeader_2x03_P2.54mm_Vertical, F.Cu at (116.5, 103.0)
- added J3: Conn_01x04, Connector_Molex:Molex_PicoBlade_53398-0471_1x04-1MP_P1.25mm_Vertical, F.Cu at (82.2, 108.2)
- added J7: Conn_01x02, Connector_PinHeader_2.54mm:PinHeader_2x01_P2.54mm_Vertical, F.Cu at (120.5, 100.4)
- added J8: Servo, Connector_PinHeader_2.54mm:PinHeader_2x03_P2.54mm_Vertical, F.Cu at (127.0, 103.0)
- added JP3: Servo Voltage, Findersee_parts:0402_Jumper_3pin, F.Cu at (121.7, 103.4)
- added R13: 0R, Resistor_SMD:R_0603_1608Metric, B.Cu at (84.5, 144.9)
- added R14: 0R, Resistor_SMD:R_0603_1608Metric, B.Cu at (86.8, 145.8)
- added U1: ADS1115IDGS, Package_SO:TSSOP-10_3x3mm_P0.5mm, F.Cu at (72.4, 142.2)
- J15: renamed from J505; value PWR_IN -> PWR_STACK
- J6: renamed from J305; footprint Connector_PinHeader_2.54mm:PinHeader_1x03_P2.54mm_Vertical -> Connector_JST:JST_SH_BM03B-SRSS-TB_1x03-1MP_P1.00mm_Vertical
- J9: renamed from J403; value DEPTH -> Conn_01x08; footprint Connector_PinHeader_2.54mm:PinHeader_1x06_P2.54mm_Vertical -> Connector_JST:JST_SH_SM08B-SRSS-TB_1x08-1MP_P1.00mm_Horizontal
- R1: renamed from R210; value 4k7 -> 2k2
- R11: renamed from R209; value 4k7 -> 2k2
- R17: renamed from R503; value R_Small -> 10k
- R18: renamed from R504; value R_Small -> 10k
- R2: renamed from R211; value 4k7 -> 2k2
- R6: renamed from R208; value 10k -> 180k
- moved R10 13.3 mm to (78.5, 143.7), turned to 0 degrees
- moved R6 12.0 mm to (81.8, 143.7), turned to 0 degrees
- moved R2 11.5 mm to (147.8, 121.2), turned to 90 degrees
- moved R9 10.6 mm to (78.5, 142.0), turned to 0 degrees
- moved R5 9.07 mm to (81.8, 142.0), turned to 0 degrees
- moved R11 9.01 mm to (79.0, 136.0), turned to 180 degrees
- moved J1 8.55 mm to (85.3, 138.7), turned to 90 degrees
- moved R8 7.90 mm to (78.5, 140.3), turned to 0 degrees
- moved R1 7.39 mm to (147.8, 125.4)
- moved J9 7.14 mm to (75.0, 98.2), turned to -90 degrees
- moved R4 6.27 mm to (81.8, 140.3), turned to 0 degrees
- moved R7 5.71 mm to (78.5, 138.7), turned to 0 degrees
- moved R16 5.09 mm to (146.6, 138.5), turned to 0 degrees
- moved R3 3.86 mm to (81.8, 138.7), turned to 0 degrees
- moved J6 2.73 mm to (140.5, 122.3), turned to 90 degrees
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- renumbered D503 to D1, D504 to D2, H401 to H1, H402 to H2, H403 to H3, H404 to H4, J202 to J1, J401 to J10, J504 to J12, J503 to J13, J502 to J14, J203 to J2, J204 to J4, J301 to J5, Q503 to Q1, Q504 to Q2, R204 to R10, R303 to R12, R401 to R15, R402 to R16, R205 to R3, R206 to R4, R207 to R5, R201 to R7, R202 to R8, R203 to R9, U301 to U2
Connections:
- net Net-(D503-Pad1) renamed /Power + FETs/CH1 OUT
- net Net-(D504-Pad1) renamed /Power + FETs/CH2 OUT
- net Net-(J202-Pad1) renamed /Connectors/CURRENT
- net Net-(J202-Pad7) renamed /Connectors/MOT VOLT
- J10 pad 3: unconnected-(J401-Pad3) -> /Connectors/RPI_I2C_SDA
- J10 pad 5: unconnected-(J401-Pad5) -> /Connectors/RPI_I2C_SCL
- J13 pad 3: +VSW -> Net-(J13-Pin_3)
- J14 pad 1: +VSW -> /Power + FETs/CH1 FUSED
- J14 pad 3: +VSW -> /Power + FETs/CH2 FUSED
- J5 pad 2: Net-(J301-Pad2) -> Net-(J5-Pin_2)
- J5 pad 3: Net-(J301-Pad3) -> Net-(J5-Pin_3)
- J9 pad 1: /Connectors/DL -> Net-(J9-Pin_1)
- J9 pad 2: +5V -> GND
- J9 pad 3: GND -> unconnected-(J9-Pin_3-Pad3)
- J9 pad 4: /Connectors/DR -> Net-(J9-Pin_4)
- J9 pad 5: +5V -> /Connectors/REAR LEFT
- J9 pad 6: GND -> /Connectors/REAR RIGHT
- Q1 pad 4: /MCU/PWM_3 -> /MCU/PWM_1
- Q2 pad 4: /MCU/PWM_4 -> /MCU/PWM_2
- R11 pad 1: Net-(J201-Pad5) -> VDD
- R11 pad 2: VDD -> Net-(U1-ADDR)
- R17 pad 1: /MCU/PWM_3 -> /MCU/PWM_1
- R18 pad 1: /MCU/PWM_4 -> /MCU/PWM_2
- U2 pad 10: Net-(J301-Pad3) -> /Connectors/RPI_I2C_SCL
- U2 pad 21: /MCU/PWM_4 -> /MCU/PWM_2
- U2 pad 22: /MCU/PWM_3 -> /MCU/PWM_1
- U2 pad 24: /MCU/PWM_2 -> /Connectors/Servo 1
- U2 pad 25: /MCU/PWM_1 -> /Connectors/Servo 2
- U2 pad 26: unconnected-(U301-Pad26) -> /Connectors/DEPTH LEFT
- U2 pad 27: /MCU/ADS_RDY -> /Connectors/DEPTH RIGHT
- U2 pad 29: /Connectors/PR -> /Connectors/REAR LEFT
- U2 pad 31: /Connectors/PL -> /Connectors/REAR RIGHT
- U2 pad 32: /Connectors/DR -> /Connectors/FRONT LEFT
- U2 pad 34: /Connectors/DL -> /Connectors/FRONT RIGHT
- U2 pad 4: unconnected-(U301-Pad4) -> Net-(J5-Pin_3)
- U2 pad 41: /Connectors/USB + -> unconnected-(U2-TP3(DP)-Pad41)
- U2 pad 42: /Connectors/USB - -> unconnected-(U2-TP2(DM)-Pad42)
- U2 pad 43: GND -> unconnected-(U2-TP1(GND)-Pad43)
- U2 pad 5: unconnected-(U301-Pad5) -> Net-(J5-Pin_2)
- U2 pad 6: unconnected-(U301-Pad6) -> /MCU/ADS_RDY
- U2 pad 9: Net-(J301-Pad2) -> /Connectors/RPI_I2C_SDA
Routing:
- net Net-(J9-Pin_1): track 0.00 -> 103.2 mm, vias 0 -> 1
- net Net-(J9-Pin_4): track 0.00 -> 90.7 mm, vias 0 -> 1
- net /Sensors/SCL: track 74.3 -> 135.0 mm, vias 2 -> 5
- net VDD: track 72.2 -> 15.7 mm, vias 16 -> 17
- net /Connectors/PR: track 53.4 -> 0.00 mm
- net /Sensors/SDA: track 85.7 -> 137.6 mm, vias 0 -> 2
- net /Connectors/PL: track 49.6 -> 0.00 mm
- net /Connectors/REAR LEFT: track 0.00 -> 46.3 mm
- net /Connectors/RPI_I2C_SDA: track 0.00 -> 44.7 mm, vias 0 -> 1
- net /Connectors/REAR RIGHT: track 0.00 -> 41.2 mm
- net /Connectors/RPI_I2C_SCL: track 0.00 -> 39.6 mm, vias 0 -> 1
- net /Connectors/DL: track 37.2 -> 0.00 mm
- net /Connectors/FRONT LEFT: track 0.00 -> 37.0 mm
- net /Connectors/DR: track 33.9 -> 0.00 mm
- net /Connectors/FRONT RIGHT: track 0.00 -> 31.2 mm
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- added copper zone on B.Cu, net +VSW
- added copper zone on B.Cu, net /Power + FETs/CH1 FUSED
- added copper zone on B.Cu, net /Power + FETs/CH2 FUSED
- added copper zone on In2.Cu, net VDD
- removed copper zone on F.Cu, net Net-(D501-Pad1)
- removed copper zone on F.Cu, net Net-(D502-Pad1)
- removed copper zone on B.Cu, net VDD
Other:
- outline, holes or cut-outs redrawn
- board text added: "FUSED"
- board text added: "Findersee 05/26 REV ${REVISION}"
- board text added: "NEG"
- board text added: "PWM"
- board text removed: "1"
- board text removed: "11"
- board text removed: "13"
- board text removed: "5"
- board text removed: "A"
- board text removed: "A/V"
- board text removed: "ACT"
- board text removed: "CAMERA"
- board text removed: "DEPTH"
- board text removed: "DISPLAY"
- board text removed: "E"
- board text removed: "ETHERNET"
- board text removed: "Findersee 03/23 REV 1"
- board text removed: "GPIO"
- board text removed: "HDMI"
- board text removed: "IN CHINA"
- board text removed: "K"
- board text removed: "LEFT"
- board text removed: "Made in the UK"
- board text removed: "N"
- board text removed: "PCB MADE"
- board text removed: "PEN"
- board text removed: "PROPULSION"
- board text removed: "PWR IN"
- board text removed: "PoE"
- board text removed: "RIGHT"
- board text removed: "RUN"
- board text removed: "Raspberry Pi 3 Model B"
- board text removed: "S + - S + -"
- board text removed: "TOP ASSEMBLY"
- board text removed: "TOP LEGEND"
- board text removed: "USB"
- board text removed: "c Raspberry Pi 2017"

Commit message: Manufacturing commit
Routing:
- net +5V: track 28.1 -> 14.7 mm, vias 11 -> 10
- net /Sensors/SCL: track 135.0 -> 126.0 mm, vias 5 -> 4
- net /Sensors/SDA: track 137.6 -> 128.6 mm
