File: electronics/RovHat/RovHat.kicad_sch (KiCad schematic)
At the start: 0 parts

Commit message: Fabrication commit
Other:
- sheet MCU ports: added ADS_RDY; removed none
- sheet Sensors ports: added ADS_RDY; removed none
Changed lines of the file:
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@@
+    (stroke (width 0) (type default) (color 0 0 0 0))
+  )
+  (wire (pts (xy 144.78 44.45) (xy 266.7 44.45))
     (stroke (width 0) (type default) (color 0 0 0 0))
   )
@@
       (effects (font (size 1.27 1.27)) (justify right))
     )
+    (pin "ADS_RDY" input (at 144.78 44.45 0)
+      (effects (font (size 1.27 1.27)) (justify right))
+    )
   )
   (sheet (at 266.7 96.52) (size 49.53 50.8) (fields_autoplaced)
@@
     )
     (pin "LSM_INT2" output (at 266.7 74.93 180)
+      (effects (font (size 1.27 1.27)) (justify left))
+    )
+    (pin "ADS_RDY" output (at 266.7 44.45 180)
       (effects (font (size 1.27 1.27)) (justify left))
     )
@@
       (reference "#FLG0103") (unit 1) (value "PWR_FLAG") (footprint "")
     )
-    (path "/ac5eb4a7-a387-48d6-b4f5-8a76d938534b/19cd669a-4c1b-473a-b3f0-d9f48828f632"
-      (reference "#FLG0104") (unit 1) (value "PWR_FLAG") (footprint "")
-    )
-    (path "/ac5eb4a7-a387-48d6-b4f5-8a76d938534b/37a1b69b-8bd0-4989-8b0a-8868e66416a5"
-      (reference "#PWR0101") (unit 1) (value "+3.3VA") (footprint "")
-    )
-    (path "/ac5eb4a7-a387-48d6-b4f5-8a76d938534b/1b8e11a6-d4b2-498b-bea0-3d795199eb91"
-      (reference "#PWR0102") (unit 1) (value "VDD") (footprint "")
-    )
-    (path "/ac5eb4a7-a387-48d6-b4f5-8a76d938534b/7cd4cdd1-5dd2-477d-9f40-7d25742c3ad0"
-      (reference "#PWR0103") (unit 1) (value "GND") (footprint "")
-    )
-    (path "/ac5eb4a7-a387-48d6-b4f5-8a76d938534b/0cc51f7e-0703-4ebb-bb7e-5655054a9bcb"
-      (reference "#PWR0104") (unit 1) (value "GND") (footprint "")
+    (path "/ac5eb4a7-a387-48d6-b4f5-8a76d938534b/e1d5cb1f-96ca-46e5-bc6f-16b434bf08b6"
+      (reference "#PWR0101") (unit 1) (value "VDD") (footprint "")
+    )
+    (path "/ac5eb4a7-a387-48d6-b4f5-8a76d938534b/0aa5114b-1ba6-4a33-a3ec-873121403519"
+      (reference "#PWR0102") (unit 1) (value "+5V") (footprint "")
     )
     (path "/ac5eb4a7-a387-48d6-b4f5-8a76d938534b/9a536964-d071-415f-addc-5ab8dab2c04a"
@@
       (reference "#PWR0129") (unit 1) (value "VBUS") (footprint "")
     )
-    (path "/ac5eb4a7-a387-48d6-b4f5-8a76d938534b/2ed2429b-3346-4e05-a839-5c69e0f0f9d8"
-      (reference "#PWR0201") (unit 1) (value "+3.3VA") (footprint "")
+    (path "/ac5eb4a7-a387-48d6-b4f5-8a76d938534b/fd9d1416-0e51-45d9-b5de-e7af208153c3"
+      (reference "#PWR0202") (unit 1) (value "VDD") (footprint "")
     )
     (path "/ac5eb4a7-a387-48d6-b4f5-8a76d938534b/254c7cd0-eb1e-44b3-b26a-d8b6f71faa2f"
@@
       (reference "#PWR0207") (unit 1) (value "GND") (footprint "")
     )
+    (path "/0a21e7d0-6c69-4634-b2b6-f0d0223d8049/658a1765-0852-4475-8820-99a161baa0d8"
+      (reference "#PWR0301") (unit 1) (value "GND") (footprint "")
+    )
     (path "/0a21e7d0-6c69-4634-b2b6-f0d0223d8049/68f7e376-0e30-4699-a761-295d29781a5f"
       (reference "#PWR0304") (unit 1) (value "+5V") (footprint "")
@@
       (reference "#PWR0502") (unit 1) (value "GND") (footprint "")
     )
-    (path "/ac5eb4a7-a387-48d6-b4f5-8a76d938534b/31476c52-21e0-4b78-b5b3-f6e0efc129b3"
-      (reference "C201") (unit 1) (value "1u") (footprint "Capacitor_SMD:C_0402_1005Metric")
-    )
-    (path "/ac5eb4a7-a387-48d6-b4f5-8a76d938534b/e8ce1049-094c-4def-afd2-aceed6d3f1b8"
-      (reference "C202") (unit 1) (value "1u") (footprint "Capacitor_SMD:C_0603_1608Metric")
-    )
-    (path "/ac5eb4a7-a387-48d6-b4f5-8a76d938534b/f9c216d6-c5d1-43b4-9020-ec5f30d8199a"
-      (reference "FB201") (unit 1) (value "600R@100M") (footprint "Inductor_SMD:L_0805_2012Metric")
+    (path "/212ae4ce-78ca-42fb-a0a9-9e7afe94e4f9/f87f3091-786f-40ba-a8f4-17e8e2de9322"
+      (reference "#PWR0503") (unit 1) (value "+VSW") (footprint "")
+    )
+    (path "/212ae4ce-78ca-42fb-a0a9-9e7afe94e4f9/d0894518-9b75-4b48-908e-aea66a40eb2b"
+      (reference "#PWR0504") (unit 1) (value "GND") (footprint "")
     )
     (path "/d0328239-535b-4cf1-98be-6519c44fecfc/d0522802-41e1-4aa4-bdd1-cf465949a1f4"
@@
     )
     (path "/ac5eb4a7-a387-48d6-b4f5-8a76d938534b/50df8fa0-ee2a-4112-85b7-c22bb6e6d9c5"
-      (reference "J201") (unit 1) (value "Conn_01x10") (footprint "Connector_PinHeader_2.54mm:PinHeader_1x10_P2.54mm_Vertical")
+      (reference "J201") (unit 1) (value "ADS1115") (footprint "Connector_PinHeader_2.54mm:PinHeader_1x10_P2.54mm_Vertical")
     )
     (path "/ac5eb4a7-a387-48d6-b4f5-8a76d938534b/79e86705-4e6f-4cfb-ad1c-b2ff2c94d675"
-      (reference "J202") (unit 1) (value "Conn_02x04_Odd_Even") (footprint "Connector_PinHeader_2.54mm:PinHeader_2x04_P2.54mm_Vertical")
+      (reference "J202") (unit 1) (value "ANALOG INPUT") (footprint "Connector_PinHeader_2.54mm:PinHeader_2x04_P2.54mm_Vertical")
     )
     (path "/ac5eb4a7-a387-48d6-b4f5-8a76d938534b/7dcb4044-e8c8-4a51-8ad5-63177668dbe8"
-      (reference "J203") (unit 1) (value "Conn_01x10") (footprint "Connector_PinHeader_2.54mm:PinHeader_1x10_P2.54mm_Vertical")
+      (reference "J203") (unit 1) (value "GYRO") (footprint "Connector_PinHeader_2.54mm:PinHeader_1x10_P2.54mm_Vertical")
+    )
+    (path "/0a21e7d0-6c69-4634-b2b6-f0d0223d8049/9faf5cae-23c2-45fa-b08c-c9b7bfd06b38"
+      (reference "J301") (unit 1) (value "PWM_OUT") (footprint "Connector_PinHeader_2.54mm:PinHeader_1x03_P2.54mm_Vertical")
     )
     (path "/0a21e7d0-6c69-4634-b2b6-f0d0223d8049/6ee1865a-79a4-421e-9e9b-877dedddec70"
@@
       (reference "J507") (unit 1) (value "PWR OUT") (footprint "Connector_PinHeader_2.54mm:PinHeader_1x02_P2.54mm_Vertical")
     )
+    (path "/212ae4ce-78ca-42fb-a0a9-9e7afe94e4f9/9d6bdb57-0b7f-44c2-8c53-caf6f843f96c"
+      (reference "J508") (unit 1) (value "PWR OUT2") (footprint "Connector_Phoenix_MC:PhoenixContact_MCV_1,5_2-G-3.5_1x02_P3.50mm_Vertical")
+    )
     (path "/212ae4ce-78ca-42fb-a0a9-9e7afe94e4f9/ea3205bd-63c2-4b68-8f79-e7d557f0c3ea"
       (reference "Q501") (unit 1) (value "IRF7403") (footprint "Package_SO:SOIC-8_3.9x4.9mm_P1.27mm")
@@
     )
     (path "/ac5eb4a7-a387-48d6-b4f5-8a76d938534b/547be16a-156b-4fb7-9944-5b8f99ecfb33"
-      (reference "R201") (unit 1) (value "20k") (footprint "Resistor_SMD:R_0402_1005Metric")
+      (reference "R201") (unit 1) (value "20k") (footprint "Resistor_SMD:R_0603_1608Metric")
     )
     (path "/ac5eb4a7-a387-48d6-b4f5-8a76d938534b/d2b2391a-6447-40d9-8989-0f9b94260921"
-      (reference "R202") (unit 1) (value "20k") (footprint "Resistor_SMD:R_0402_1005Metric")
+      (reference "R202") (unit 1) (value "20k") (footprint "Resistor_SMD:R_0603_1608Metric")
     )
     (path "/ac5eb4a7-a387-48d6-b4f5-8a76d938534b/2c95787e-d13f-4996-ad28-fbc4c8edac60"
-      (reference "R203") (unit 1) (value "20k") (footprint "Resistor_SMD:R_0402_1005Metric")
+      (reference "R203") (unit 1) (value "20k") (footprint "Resistor_SMD:R_0603_1608Metric")
     )
     (path "/ac5eb4a7-a387-48d6-b4f5-8a76d938534b/b1986a92-7dd9-4305-b6db-f39e64fc10ad"
-      (reference "R204") (unit 1) (value "20k") (footprint "Resistor_SMD:R_0402_1005Metric")
+      (reference "R204") (unit 1) (value "20k") (footprint "Resistor_SMD:R_0603_1608Metric")
     )
     (path "/ac5eb4a7-a387-48d6-b4f5-8a76d938534b/d54b3f4d-4433-48df-805e-d6814983a33f"
-      (reference "R205") (unit 1) (value "10k") (footprint "Resistor_SMD:R_0402_1005Metric")
+      (reference "R205") (unit 1) (value "10k") (footprint "Resistor_SMD:R_0603_1608Metric")
     )
     (path "/ac5eb4a7-a387-48d6-b4f5-8a76d938534b/ec703c70-bfbb-446c-a6d1-dcb2f025fc2e"
-      (reference "R206") (unit 1) (value "10k") (footprint "Resistor_SMD:R_0402_1005Metric")
+      (reference "R206") (unit 1) (value "10k") (footprint "Resistor_SMD:R_0603_1608Metric")
     )
     (path "/ac5eb4a7-a387-48d6-b4f5-8a76d938534b/aa4c6a35-0fea-40d8-9c62-56227baaa7c9"
-      (reference "R207") (unit 1) (value "10k") (footprint "Resistor_SMD:R_0402_1005Metric")
+      (reference "R207") (unit 1) (value "10k") (footprint "Resistor_SMD:R_0603_1608Metric")
     )
     (path "/ac5eb4a7-a387-48d6-b4f5-8a76d938534b/85f2766e-253c-4942-8584-87dee2050f4c"
-      (reference "R208") (unit 1) (value "10k") (footprint "Resistor_SMD:R_0402_1005Metric")
+      (reference "R208") (unit 1) (value "10k") (footprint "Resistor_SMD:R_0603_1608Metric")
+    )
+    (path "/ac5eb4a7-a387-48d6-b4f5-8a76d938534b/3c5fee81-ce0b-4c72-8208-9ada2d38fdd5"
+      (reference "R209") (unit 1) (value "4k7") (footprint "Resistor_SMD:R_0603_1608Metric")
+    )
+    (path "/ac5eb4a7-a387-48d6-b4f5-8a76d938534b/fa7fd25c-e554-4803-9ab7-2eed2b71a038"
+      (reference "R210") (unit 1) (value "4k7") (footprint "Resistor_SMD:R_0603_1608Metric")
+    )
+    (path "/ac5eb4a7-a387-48d6-b4f5-8a76d938534b/6273d1ea-6f0e-4979-9a07-65fae51eb396"
+      (reference "R211") (unit 1) (value "4k7") (footprint "Resistor_SMD:R_0603_1608Metric")
     )
     (path "/0a21e7d0-6c69-4634-b2b6-f0d0223d8049/63c68d2d-6842-43df-b3ee-ec7e150c4a01"

Commit message: Fabrication commit 2
Parts:
- added H401, H402, H403, H404: MountingHole, MountingHole:MountingHole_2.7mm_M2.5, symbol Mechanical:MountingHole
Other:
- company: (none) -> Findersee
- title: (none) -> ROV RPI PICO HAT
Changed lines of the file:
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@@
 (kicad_sch (version 20211123) (generator eeschema)
   (paper "A3")
+  (title_block
+    (title "ROV RPI PICO HAT")
+    (date "2023-01-14")
+    (rev "1")
+    (company "Findersee")
+    (comment 1 "Main Block Diagram")
+  )
   (wire (pts (xy 144.78 54.61) (xy 266.7 54.61))
     (stroke (width 0) (type default) (color 0 0 0 0))
@@
   (wire (pts (xy 144.78 200.66) (xy 266.7 200.66))
     (stroke (width 0) (type default) (color 0 0 0 0))
+  )
+  (symbol (lib_id "Mechanical:MountingHole") (at 386.08 217.17 0) (unit 1)
+    (in_bom yes) (on_board yes) (fields_autoplaced)
+    (property "Reference" "H401" (id 0) (at 388.62 216.2615 0)
+      (effects (font (size 1.27 1.27)) (justify left))
+    )
+    (property "Value" "MountingHole" (id 1) (at 388.62 219.0366 0)
+      (effects (font (size 1.27 1.27)) (justify left))
+    )
+    (property "Footprint" "MountingHole:MountingHole_2.7mm_M2.5" (id 2) (at 386.08 217.17 0)
+      (effects (font (size 1.27 1.27)) hide)
+    )
+    (property "Datasheet" "~" (id 3) (at 386.08 217.17 0)
+      (effects (font (size 1.27 1.27)) hide)
+    )
+  )
+  (symbol (lib_id "Mechanical:MountingHole") (at 386.08 224.79 0) (unit 1)
+    (in_bom yes) (on_board yes) (fields_autoplaced)
+    (property "Reference" "H402" (id 0) (at 388.62 223.8815 0)
+      (effects (font (size 1.27 1.27)) (justify left))
+    )
+    (property "Value" "MountingHole" (id 1) (at 388.62 226.6566 0)
+      (effects (font (size 1.27 1.27)) (justify left))
+    )
+    (property "Footprint" "MountingHole:MountingHole_2.7mm_M2.5" (id 2) (at 386.08 224.79 0)
+      (effects (font (size 1.27 1.27)) hide)
+    )
+    (property "Datasheet" "~" (id 3) (at 386.08 224.79 0)
+      (effects (font (size 1.27 1.27)) hide)
+    )
+  )
+  (symbol (lib_id "Mechanical:MountingHole") (at 386.08 240.03 0) (unit 1)
+    (in_bom yes) (on_board yes) (fields_autoplaced)
+    (property "Reference" "H404" (id 0) (at 388.62 239.1215 0)
+      (effects (font (size 1.27 1.27)) (justify left))
+    )
+    (property "Value" "MountingHole" (id 1) (at 388.62 241.8966 0)
+      (effects (font (size 1.27 1.27)) (justify left))
+    )
+    (property "Footprint" "MountingHole:MountingHole_2.7mm_M2.5" (id 2) (at 386.08 240.03 0)
+      (effects (font (size 1.27 1.27)) hide)
+    )
+    (property "Datasheet" "~" (id 3) (at 386.08 240.03 0)
+      (effects (font (size 1.27 1.27)) hide)
+    )
+  )
+  (symbol (lib_id "Mechanical:MountingHole") (at 386.08 232.41 0) (unit 1)
+    (in_bom yes) (on_board yes) (fields_autoplaced)
+    (property "Reference" "H403" (id 0) (at 388.62 231.5015 0)
+      (effects (font (size 1.27 1.27)) (justify left))
+    )
+    (property "Value" "MountingHole" (id 1) (at 388.62 234.2766 0)
+      (effects (font (size 1.27 1.27)) (justify left))
+    )
+    (property "Footprint" "MountingHole:MountingHole_2.7mm_M2.5" (id 2) (at 386.08 232.41 0)
+      (effects (font (size 1.27 1.27)) hide)
+    )
+    (property "Datasheet" "~" (id 3) (at 386.08 232.41 0)
+      (effects (font (size 1.27 1.27)) hide)
+    )
   )
   (sheet (at 82.55 25.654) (size 62.23 220.726) (fields_autoplaced)
@@
       (reference "#PWR0504") (unit 1) (value "GND") (footprint "")
     )
-    (path "/d0328239-535b-4cf1-98be-6519c44fecfc/d0522802-41e1-4aa4-bdd1-cf465949a1f4"
+    (path "/212ae4ce-78ca-42fb-a0a9-9e7afe94e4f9/ae3bc981-dc5d-4efc-a359-2dbd858997b3"
+      (reference "D501") (unit 1) (value "MBR0550") (footprint "Diode_SMD:D_SOD-123")
+    )
+    (path "/212ae4ce-78ca-42fb-a0a9-9e7afe94e4f9/6d32de7f-8511-4acc-ae00-a355e28677f8"
+      (reference "D502") (unit 1) (value "MBR0550") (footprint "Diode_SMD:D_SOD-123")
+    )
+    (path "/212ae4ce-78ca-42fb-a0a9-9e7afe94e4f9/1d83f8fb-331a-45cf-b7e4-73d15afe4549"
+      (reference "D503") (unit 1) (value "MBR0550") (footprint "Diode_SMD:D_SOD-123")
+    )
+    (path "/212ae4ce-78ca-42fb-a0a9-9e7afe94e4f9/b7f32931-ffe5-41b6-babb-50097a414397"
+      (reference "D504") (unit 1) (value "MBR0550") (footprint "Diode_SMD:D_SOD-123")
+    )
+    (path "/02a6deef-a27e-4f78-9132-f029461a1c12"
       (reference "H401") (unit 1) (value "MountingHole") (footprint "MountingHole:MountingHole_2.7mm_M2.5")
     )
-    (path "/d0328239-535b-4cf1-98be-6519c44fecfc/825a18b0-cab3-4ca5-8fad-c014f4c769aa"
+    (path "/13b93b86-c7f7-4bd6-8395-83e3bb2ec213"
       (reference "H402") (unit 1) (value "MountingHole") (footprint "MountingHole:MountingHole_2.7mm_M2.5")
     )
-    (path "/d0328239-535b-4cf1-98be-6519c44fecfc/03237fd7-78d8-4d96-ad96-ce43adb9aa63"
+    (path "/c11d4df1-2d00-44e1-90be-b73677a9c998"
       (reference "H403") (unit 1) (value "MountingHole") (footprint "MountingHole:MountingHole_2.7mm_M2.5")
     )
-    (path "/d0328239-535b-4cf1-98be-6519c44fecfc/de7fea8d-4e42-45f2-bcd8-b104da103d2e"
+    (path "/8db2cc8d-4ba9-4c46-9a6a-2505da4c7844"
       (reference "H404") (unit 1) (value "MountingHole") (footprint "MountingHole:MountingHole_2.7mm_M2.5")
     )

Commit message: Final Version
Changed lines of the file:
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@@
     )
   )
-  (sheet (at 266.7 193.04) (size 50.8 50.8) (fields_autoplaced)
+  (sheet (at 266.7 177.8) (size 50.8 66.04) (fields_autoplaced)
     (stroke (width 0.1524) (type solid) (color 0 0 0 0))
     (fill (color 255 255 194 1.0000))
-    (property "Sheet name" "Connectors" (id 0) (at 266.7 192.3284 0)
+    (property "Sheet name" "Connectors" (id 0) (at 266.7 177.0884 0)
       (effects (font (size 1.27 1.27)) (justify left bottom))
     )
@@
   )
   (symbol_instances
-    (path "/212ae4ce-78ca-42fb-a0a9-9e7afe94e4f9/876ab51d-81be-4e3d-b934-e8be2b045c4e"
+    (path "/212ae4ce-78ca-42fb-a0a9-9e7afe94e4f9/9b85af59-f883-49f0-a4fb-3ce3c1742924"
       (reference "#FLG0101") (unit 1) (value "PWR_FLAG") (footprint "")
     )
@@
       (reference "#PWR0102") (unit 1) (value "+5V") (footprint "")
     )
+    (path "/212ae4ce-78ca-42fb-a0a9-9e7afe94e4f9/82485a7b-8104-4c24-8b9e-d0b1a9cd4d80"
+      (reference "#PWR0103") (unit 1) (value "GND") (footprint "")
+    )
+    (path "/212ae4ce-78ca-42fb-a0a9-9e7afe94e4f9/98b1528c-47de-4a4b-ac17-9a1e2a87843a"
+      (reference "#PWR0104") (unit 1) (value "+VSW") (footprint "")
+    )
     (path "/ac5eb4a7-a387-48d6-b4f5-8a76d938534b/9a536964-d071-415f-addc-5ab8dab2c04a"
       (reference "#PWR0105") (unit 1) (value "GND") (footprint "")
@@
       (reference "#PWR0112") (unit 1) (value "GND") (footprint "")
     )
-    (path "/212ae4ce-78ca-42fb-a0a9-9e7afe94e4f9/a2ebd9c3-6957-49e4-8ece-cafeb750b504"
-      (reference "#PWR0113") (unit 1) (value "+VSW") (footprint "")
-    )
     (path "/212ae4ce-78ca-42fb-a0a9-9e7afe94e4f9/e1dd61aa-e746-4e8f-8c07-870eb3bb4824"
       (reference "#PWR0114") (unit 1) (value "+VSW") (footprint "")
@@
       (reference "#PWR0115") (unit 1) (value "GND") (footprint "")
     )
-    (path "/212ae4ce-78ca-42fb-a0a9-9e7afe94e4f9/1e65f158-00e5-4382-8291-99352f9659ad"
-      (reference "#PWR0116") (unit 1) (value "+VSW") (footprint "")
-    )
     (path "/212ae4ce-78ca-42fb-a0a9-9e7afe94e4f9/48d01efe-2862-46c8-b776-75d3312c329c"
       (reference "#PWR0117") (unit 1) (value "+VSW") (footprint "")
@@
       (reference "#PWR0119") (unit 1) (value "GND") (footprint "")
     )
-    (path "/212ae4ce-78ca-42fb-a0a9-9e7afe94e4f9/2bbc7a2e-364b-426b-b695-ef57df79f744"
-      (reference "#PWR0120") (unit 1) (value "GND") (footprint "")
-    )
-    (path "/212ae4ce-78ca-42fb-a0a9-9e7afe94e4f9/7c5c5897-05da-4a53-a7fa-aef2f6dfd530"
-      (reference "#PWR0121") (unit 1) (value "+VSW") (footprint "")
-    )
     (path "/212ae4ce-78ca-42fb-a0a9-9e7afe94e4f9/f6588f1d-fa61-4e05-b84a-637e85dd9c0d"
       (reference "#PWR0122") (unit 1) (value "+5V") (footprint "")
@@
       (reference "#PWR0129") (unit 1) (value "VBUS") (footprint "")
     )
+    (path "/ac5eb4a7-a387-48d6-b4f5-8a76d938534b/cb7034e3-d777-4193-9627-5137b589596d"
+      (reference "#PWR0201") (unit 1) (value "VDD") (footprint "")
+    )
     (path "/ac5eb4a7-a387-48d6-b4f5-8a76d938534b/fd9d1416-0e51-45d9-b5de-e7af208153c3"
       (reference "#PWR0202") (unit 1) (value "VDD") (footprint "")
@@
       (reference "#PWR0207") (unit 1) (value "GND") (footprint "")
     )
+    (path "/ac5eb4a7-a387-48d6-b4f5-8a76d938534b/1644925e-e166-433d-b194-7b2a1786cc77"
+      (reference "#PWR0208") (unit 1) (value "GND") (footprint "")
+    )
     (path "/0a21e7d0-6c69-4634-b2b6-f0d0223d8049/658a1765-0852-4475-8820-99a161baa0d8"
       (reference "#PWR0301") (unit 1) (value "GND") (footprint "")
@@
       (reference "#PWR0504") (unit 1) (value "GND") (footprint "")
     )
+    (path "/212ae4ce-78ca-42fb-a0a9-9e7afe94e4f9/ccc9d90b-da4a-4e8d-ad59-1906856fc820"
+      (reference "#PWR0505") (unit 1) (value "+VSW") (footprint "")
+    )
+    (path "/212ae4ce-78ca-42fb-a0a9-9e7afe94e4f9/a8557804-ebe2-432e-90f7-e52a1abef969"
+      (reference "#PWR0506") (unit 1) (value "+VSW") (footprint "")
+    )
     (path "/212ae4ce-78ca-42fb-a0a9-9e7afe94e4f9/ae3bc981-dc5d-4efc-a359-2dbd858997b3"
       (reference "D501") (unit 1) (value "MBR0550") (footprint "Diode_SMD:D_SOD-123")
@@
       (reference "J203") (unit 1) (value "GYRO") (footprint "Connector_PinHeader_2.54mm:PinHeader_1x10_P2.54mm_Vertical")
     )
+    (path "/ac5eb4a7-a387-48d6-b4f5-8a76d938534b/c1091f2c-62d0-46ef-9c1c-bcb2a9bf0032"
+      (reference "J204") (unit 1) (value "I2C EXPAND") (footprint "Connector_PinHeader_2.54mm:PinHeader_1x04_P2.54mm_Vertical")
+    )
     (path "/0a21e7d0-6c69-4634-b2b6-f0d0223d8049/9faf5cae-23c2-45fa-b08c-c9b7bfd06b38"
       (reference "J301") (unit 1) (value "PWM_OUT") (footprint "Connector_PinHeader_2.54mm:PinHeader_1x03_P2.54mm_Vertical")
@@
       (reference "J404") (unit 1) (value "PROPULSION") (footprint "Connector_PinHeader_2.54mm:PinHeader_1x06_P2.54mm_Vertical")
     )
-    (path "/212ae4ce-78ca-42fb-a0a9-9e7afe94e4f9/766c0a7c-fe31-4dc7-910a-3155685bbae7"
-      (reference "J501") (unit 1) (value "OUT1") (footprint "Connector_Phoenix_MC:PhoenixContact_MCV_1,5_2-G-3.5_1x02_P3.50mm_Vertical")
-    )
-    (path "/212ae4ce-78ca-42fb-a0a9-9e7afe94e4f9/e2783a59-ade3-402d-a7f0-a773422eb380"
-      (reference "J502") (unit 1) (value "OUT2") (footprint "Connector_Phoenix_MC:PhoenixContact_MCV_1,5_2-G-3.5_1x02_P3.50mm_Vertical")
-    )
-    (path "/212ae4ce-78ca-42fb-a0a9-9e7afe94e4f9/cc20f63e-6b7a-474c-a3ec-5fbbd487587b"
-      (reference "J503") (unit 1) (value "OUT3") (footprint "Connector_Phoenix_MC:PhoenixContact_MCV_1,5_2-G-3.5_1x02_P3.50mm_Vertical")
+    (path "/212ae4ce-78ca-42fb-a0a9-9e7afe94e4f9/567954bd-6203-450b-8790-c3b2c2a0f6aa"
+      (reference "J501") (unit 1) (value "OUT1") (footprint "Connector_Phoenix_MC:PhoenixContact_MCV_1,5_4-G-3.5_1x04_P3.50mm_Vertical")
+    )
+    (path "/212ae4ce-78ca-42fb-a0a9-9e7afe94e4f9/e40a658e-5095-49ef-906c-b2d9ebca28bb"
+      (reference "J502") (unit 1) (value "OUT2") (footprint "Connector_Phoenix_MC:PhoenixContact_MCV_1,5_4-G-3.5_1x04_P3.50mm_Vertical")
+    )
+    (path "/212ae4ce-78ca-42fb-a0a9-9e7afe94e4f9/3409ff77-6ba7-4502-9966-0e6290fba3d7"
+      (reference "J503") (unit 1) (value "PWR") (footprint "Connector_Phoenix_MC:PhoenixContact_MCV_1,5_4-G-3.5_1x04_P3.50mm_Vertical")
     )
     (path "/212ae4ce-78ca-42fb-a0a9-9e7afe94e4f9/8a19a795-79df-4239-aa69-948cbf817130"
       (reference "J504") (unit 1) (value "5V IN") (footprint "Connector_PinHeader_2.54mm:PinHeader_1x02_P2.54mm_Vertical")
     )
-    (path "/212ae4ce-78ca-42fb-a0a9-9e7afe94e4f9/7d750c27-6f9f-4d5f-b423-f7206a241e7c"
-      (reference "J505") (unit 1) (value "OUT4") (footprint "Connector_Phoenix_MC:PhoenixContact_MCV_1,5_2-G-3.5_1x02_P3.50mm_Vertical")
-    )
-    (path "/212ae4ce-78ca-42fb-a0a9-9e7afe94e4f9/df3d935e-3f37-45a4-9464-ebcef36158f4"
-      (reference "J506") (unit 1) (value "PWR IN") (footprint "Connector_Phoenix_MC:PhoenixContact_MCV_1,5_2-G-3.5_1x02_P3.50mm_Vertical")
-    )
-    (path "/212ae4ce-78ca-42fb-a0a9-9e7afe94e4f9/c72eadd1-e81d-4a94-822c-8d2f3a52b184"
-      (reference "J507") (unit 1) (value "PWR OUT") (footprint "Connector_PinHeader_2.54mm:PinHeader_1x02_P2.54mm_Vertical")
-    )
-    (path "/212ae4ce-78ca-42fb-a0a9-9e7afe94e4f9/9d6bdb57-0b7f-44c2-8c53-caf6f843f96c"
-      (reference "J508") (unit 1) (value "PWR OUT2") (footprint "Connector_Phoenix_MC:PhoenixContact_MCV_1,5_2-G-3.5_1x02_P3.50mm_Vertical")
+    (path "/212ae4ce-78ca-42fb-a0a9-9e7afe94e4f9/c8141d23-80b7-41ab-8d00-06dce93485de"
+      (reference "J505") (unit 1) (value "PWR_IN") (footprint "Connector_PinHeader_2.54mm:PinHeader_2x02_P2.54mm_Vertical")
     )
     (path "/212ae4ce-78ca-42fb-a0a9-9e7afe94e4f9/ea3205bd-63c2-4b68-8f79-e7d557f0c3ea"
@@
       (reference "R303") (unit 1) (value "10k") (footprint "Resistor_SMD:R_0603_1608Metric")
     )
+    (path "/d0328239-535b-4cf1-98be-6519c44fecfc/2fa6ccb3-a1fe-47a2-9882-57b873dc7873"
+      (reference "R401") (unit 1) (value "0R") (footprint "Resistor_SMD:R_0603_1608Metric")
+    )
+    (path "/d0328239-535b-4cf1-98be-6519c44fecfc/277bc8d1-0224-40f2-a4b3-cff612ff230d"
+      (reference "R402") (unit 1) (value "0R") (footprint "Resistor_SMD:R_0603_1608Metric")
+    )
     (path "/212ae4ce-78ca-42fb-a0a9-9e7afe94e4f9/20f0820b-6761-4c84-b80e-935c5d0ce68e"
