File: electronics/RovHat/RovHat.kicad_sch (KiCad schematic)
At the start: 4 parts

Commit message: Multiple fixes
Parts:
- renumbered H401 to H1, H402 to H2, H403 to H3, H404 to H4
Other:
- sheet Connectors ports: added CURRENT, DEPTH LEFT, DEPTH RIGHT, FRONT LEFT, FRONT RIGHT, MOT VOLT, REAR LEFT, REAR RIGHT, RPI_I2C_SCL, RPI_I2C_SDA, Servo 1, Servo 2; removed DL, DR, PL, PR, USB +, USB -
- sheet MCU ports: added DEPTH LEFT, DEPTH RIGHT, FRONT LEFT, FRONT RIGHT, REAR LEFT, REAR RIGHT, RPI_I2C_SCL, RPI_I2C_SDA, Servo 1, Servo 2; removed PIO1, PIO2, PIO3, PIO4, PWM_3, PWM_4, USB_D+, USB_D-
- sheet Power + FETs ports: added none; removed CH3, CH4
- sheet Sensors ports: added Current, MOT VOLT, RPI_SCL, RPI_SDA; removed none
