File: electronics/RovHat/power.kicad_sch (KiCad schematic)
At the start: 15 parts, among them J501 OUT1, J502 OUT2, J503 OUT3, J504 5V IN, J505 OUT4, J506 PWR IN, J507 PWR OUT, Q501 AOD508, Q502 AOD508, Q503 AOD508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

Commit message: Layout Done first level
Parts:
- removed Q501, Q502, Q503, Q504: AOD508, Package_TO_SOT_SMD:TO-252-2, symbol Findersee_parts:AOD508
- added Q501, Q502, Q503, Q504: IRF7403, Package_SO:SOIC-8_3.9x4.9mm_P1.27mm, symbol Transistor_FET:IRF7403
Connections:
- net CH1: now also Q501.4 (G)
- net CH2: now also Q502.4 (G)
- net CH3: now also Q503.4 (G)
- net CH4: now also Q504.4 (G)
- net GND: now also Q501.1 (S), Q501.2 (S), Q501.3 (S), Q502.1 (S), Q502.2 (S), Q502.3 (S), Q503.1 (S), Q503.2 (S), Q503.3 (S), Q504.1 (S), Q504.2 (S), Q504.3 (S)
- net at J501.2 (Pin_2): now also Q501.5 (D), Q501.6 (D), Q501.7 (D), Q501.8 (D)
- net at J502.2 (Pin_2): now also Q502.5 (D), Q502.6 (D), Q502.7 (D), Q502.8 (D)
- net at J503.2 (Pin_2): now also Q503.5 (D), Q503.6 (D), Q503.7 (D), Q503.8 (D)
- net at J505.2 (Pin_2): now also Q504.5 (D), Q504.6 (D), Q504.7 (D), Q504.8 (D)

Commit message: Fabrication commit
Parts:
- added J508: PWR OUT2, Connector_Phoenix_MC:PhoenixContact_MCV_1,5_2-G-3.5_1x02_P3.50mm_Vertical, symbol Connector_Generic:Conn_01x02
Connections:
- net +VSW: now also J508.1 (Pin_1)
- net GND: now also J508.2 (Pin_2)
Other:
- moved on the sheet: J507
Changed lines of the file:
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@@
     (stroke (width 0) (type default) (color 0 0 0 0))
   )
-  (wire (pts (xy 250.19 105.41) (xy 250.19 110.49))
+  (wire (pts (xy 250.19 104.14) (xy 250.19 109.22))
     (stroke (width 0) (type default) (color 0 0 0 0))
   )
@@
     (stroke (width 0) (type default) (color 0 0 0 0))
   )
+  (wire (pts (xy 213.36 104.14) (xy 213.36 109.22))
+    (stroke (width 0) (type default) (color 0 0 0 0))
+  )
   (wire (pts (xy 241.3 85.09) (xy 241.3 87.63))
     (stroke (width 0) (type default) (color 0 0 0 0))
@@
     (stroke (width 0) (type default) (color 0 0 0 0))
   )
+  (wire (pts (xy 213.36 111.76) (xy 213.36 115.57))
+    (stroke (width 0) (type default) (color 0 0 0 0))
+  )
   (wire (pts (xy 250.19 139.7) (xy 250.19 143.51))
     (stroke (width 0) (type default) (color 0 0 0 0))
@@
     (stroke (width 0) (type default) (color 0 0 0 0))
   )
-  (wire (pts (xy 250.19 113.03) (xy 250.19 116.84))
+  (wire (pts (xy 250.19 111.76) (xy 250.19 115.57))
     (stroke (width 0) (type default) (color 0 0 0 0))
   )
@@
     (stroke (width 0) (type default) (color 0 0 0 0))
   )
+  (wire (pts (xy 217.17 111.76) (xy 213.36 111.76))
+    (stroke (width 0) (type default) (color 0 0 0 0))
+  )
   (wire (pts (xy 229.87 82.55) (xy 229.87 85.09))
     (stroke (width 0) (type default) (color 0 0 0 0))
   )
-  (wire (pts (xy 254 113.03) (xy 250.19 113.03))
+  (wire (pts (xy 254 111.76) (xy 250.19 111.76))
     (stroke (width 0) (type default) (color 0 0 0 0))
   )
@@
     (stroke (width 0) (type default) (color 0 0 0 0))
   )
-  (wire (pts (xy 254 110.49) (xy 250.19 110.49))
+  (wire (pts (xy 217.17 109.22) (xy 213.36 109.22))
+    (stroke (width 0) (type default) (color 0 0 0 0))
+  )
+  (wire (pts (xy 254 109.22) (xy 250.19 109.22))
     (stroke (width 0) (type default) (color 0 0 0 0))
   )
@@
     (pin "1")
   )
+  (symbol (lib_id "Connector_Generic:Conn_01x02") (at 222.25 109.22 0) (unit 1)
+    (in_bom yes) (on_board yes) (fields_autoplaced)
+    (property "Reference" "J508" (id 0) (at 224.282 109.5815 0)
+      (effects (font (size 1.27 1.27)) (justify left))
+    )
+    (property "Value" "PWR OUT2" (id 1) (at 224.282 112.3566 0)
+      (effects (font (size 1.27 1.27)) (justify left))
+    )
+    (property "Footprint" "Connector_Phoenix_MC:PhoenixContact_MCV_1,5_2-G-3.5_1x02_P3.50mm_Vertical" (id 2) (at 222.25 109.22 0)
+      (effects (font (size 1.27 1.27)) hide)
+    )
+    (property "Datasheet" "~" (id 3) (at 222.25 109.22 0)
+      (effects (font (size 1.27 1.27)) hide)
+    )
+    (pin "1")
+    (pin "2")
+  )
   (symbol (lib_id "power:GND") (at 139.7 87.63 0) (unit 1)
     (in_bom yes) (on_board yes) (fields_autoplaced)
@@
     (pin "1")
   )
-  (symbol (lib_id "power:+VSW") (at 250.19 105.41 0) (unit 1)
-    (in_bom yes) (on_board yes) (fields_autoplaced)
-    (property "Reference" "#PWR0501" (id 0) (at 250.19 109.22 0)
-      (effects (font (size 1.27 1.27)) hide)
-    )
-    (property "Value" "+VSW" (id 1) (at 250.19 101.8055 0))
-    (property "Footprint" "" (id 2) (at 250.19 105.41 0)
-      (effects (font (size 1.27 1.27)) hide)
-    )
-    (property "Datasheet" "" (id 3) (at 250.19 105.41 0)
+  (symbol (lib_id "power:+VSW") (at 250.19 104.14 0) (unit 1)
+    (in_bom yes) (on_board yes) (fields_autoplaced)
+    (property "Reference" "#PWR0501" (id 0) (at 250.19 107.95 0)
+      (effects (font (size 1.27 1.27)) hide)
+    )
+    (property "Value" "+VSW" (id 1) (at 250.19 100.5355 0))
+    (property "Footprint" "" (id 2) (at 250.19 104.14 0)
+      (effects (font (size 1.27 1.27)) hide)
+    )
+    (property "Datasheet" "" (id 3) (at 250.19 104.14 0)
       (effects (font (size 1.27 1.27)) hide)
     )
@@
     (pin "1")
   )
-  (symbol (lib_id "Connector_Generic:Conn_01x02") (at 259.08 110.49 0) (unit 1)
-    (in_bom yes) (on_board yes) (fields_autoplaced)
-    (property "Reference" "J507" (id 0) (at 261.112 110.8515 0)
-      (effects (font (size 1.27 1.27)) (justify left))
-    )
-    (property "Value" "PWR OUT" (id 1) (at 261.112 113.6266 0)
-      (effects (font (size 1.27 1.27)) (justify left))
-    )
-    (property "Footprint" "Connector_PinHeader_2.54mm:PinHeader_1x02_P2.54mm_Vertical" (id 2) (at 259.08 110.49 0)
-      (effects (font (size 1.27 1.27)) hide)
-    )
-    (property "Datasheet" "~" (id 3) (at 259.08 110.49 0)
+  (symbol (lib_id "Connector_Generic:Conn_01x02") (at 259.08 109.22 0) (unit 1)
+    (in_bom yes) (on_board yes) (fields_autoplaced)
+    (property "Reference" "J507" (id 0) (at 261.112 109.5815 0)
+      (effects (font (size 1.27 1.27)) (justify left))
+    )
+    (property "Value" "PWR OUT" (id 1) (at 261.112 112.3566 0)
+      (effects (font (size 1.27 1.27)) (justify left))
+    )
+    (property "Footprint" "Connector_PinHeader_2.54mm:PinHeader_1x02_P2.54mm_Vertical" (id 2) (at 259.08 109.22 0)
+      (effects (font (size 1.27 1.27)) hide)
+    )
+    (property "Datasheet" "~" (id 3) (at 259.08 109.22 0)
       (effects (font (size 1.27 1.27)) hide)
     )
@@
     (pin "1")
     (pin "2")
+  )
+  (symbol (lib_id "power:GND") (at 213.36 115.57 0) (unit 1)
+    (in_bom yes) (on_board yes) (fields_autoplaced)
+    (property "Reference" "#PWR0504" (id 0) (at 213.36 121.92 0)
+      (effects (font (size 1.27 1.27)) hide)
+    )
+    (property "Value" "GND" (id 1) (at 213.36 120.1325 0))
+    (property "Footprint" "" (id 2) (at 213.36 115.57 0)
+      (effects (font (size 1.27 1.27)) hide)
+    )
+    (property "Datasheet" "" (id 3) (at 213.36 115.57 0)
+      (effects (font (size 1.27 1.27)) hide)
+    )
+    (pin "1")
   )
   (symbol (lib_id "Transistor_FET:IRF7403") (at 137.16 76.2 0) (unit 1)
@@
     (pin "8")
   )
-  (symbol (lib_id "power:GND") (at 250.19 116.84 0) (unit 1)
-    (in_bom yes) (on_board yes) (fields_autoplaced)
-    (property "Reference" "#PWR0502" (id 0) (at 250.19 123.19 0)
-      (effects (font (size 1.27 1.27)) hide)
-    )
-    (property "Value" "GND" (id 1) (at 250.19 121.4025 0))
-    (property "Footprint" "" (id 2) (at 250.19 116.84 0)
-      (effects (font (size 1.27 1.27)) hide)
-    )
-    (property "Datasheet" "" (id 3) (at 250.19 116.84 0)
+  (symbol (lib_id "power:GND") (at 250.19 115.57 0) (unit 1)
+    (in_bom yes) (on_board yes) (fields_autoplaced)
+    (property "Reference" "#PWR0502" (id 0) (at 250.19 121.92 0)
+      (effects (font (size 1.27 1.27)) hide)
+    )
+    (property "Value" "GND" (id 1) (at 250.19 120.1325 0))
+    (property "Footprint" "" (id 2) (at 250.19 115.57 0)
+      (effects (font (size 1.27 1.27)) hide)
+    )
+    (property "Datasheet" "" (id 3) (at 250.19 115.57 0)
       (effects (font (size 1.27 1.27)) hide)
     )
@@
       (effects (font (size 1.27 1.27)) hide)
     )
+    (pin "1")
+  )
+  (symbol (lib_id "power:+VSW") (at 213.36 104.14 0) (unit 1)
+    (in_bom yes) (on_board yes) (fields_autoplaced)
+    (property "Reference" "#PWR0503" (id 0) (at 213.36 107.95 0)
+      (effects (font (size 1.27 1.27)) hide)
+    )
+    (property "Value" "+VSW" (id 1) (at 213.36 100.5355 0))
+    (property "Footprint" "" (id 2) (at 213.36 104.14 0)
+      (effects (font (size 1.27 1.27)) hide)
+    )
+    (property "Datasheet" "" (id 3) (at 213.36 104.14 0)
+      (effects (font (size 1.27 1.27)) hide)
+    )

Commit message: Fabrication commit 2
Parts:
- added D501, D502, D503, D504: MBR0550, Diode_SMD:D_SOD-123, symbol Diode:MBR0550
Connections:
- net GND: now also D501.2 (A), D502.2 (A), D503.2 (A), D504.2 (A)
- net at J505.2 (Pin_2), Q504.5 (D), Q504.6 (D)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: now also D504.1 (K)
- net at J503.2 (Pin_2), Q503.5 (D), Q503.6 (D)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: now also D503.1 (K)
- net at J501.2 (Pin_2), Q501.5 (D), Q501.6 (D)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: now also D501.1 (K)
- net at J502.2 (Pin_2), Q502.5 (D), Q502.6 (D)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: now also D502.1 (K)
Other:
- company: (none) -> Findersee
- title: (none) -> ROV RPI PICO HAT
- moved on the sheet: J508

Commit message: Final Version
Parts:
- removed J501: OUT1, Connector_Phoenix_MC:PhoenixContact_MCV_1,5_2-G-3.5_1x02_P3.50mm_Vertical, symbol Connector_Generic:Conn_01x02
- removed J502: OUT2, Connector_Phoenix_MC:PhoenixContact_MCV_1,5_2-G-3.5_1x02_P3.50mm_Vertical, symbol Connector_Generic:Conn_01x02
- removed J503: OUT3, Connector_Phoenix_MC:PhoenixContact_MCV_1,5_2-G-3.5_1x02_P3.50mm_Vertical, symbol Connector_Generic:Conn_01x02
- removed J505: OUT4, Connector_Phoenix_MC:PhoenixContact_MCV_1,5_2-G-3.5_1x02_P3.50mm_Vertical, symbol Connector_Generic:Conn_01x02
- removed J506: PWR IN, Connector_Phoenix_MC:PhoenixContact_MCV_1,5_2-G-3.5_1x02_P3.50mm_Vertical, symbol Connector_Generic:Conn_01x02
- removed J507: PWR OUT, Connector_PinHeader_2.54mm:PinHeader_1x02_P2.54mm_Vertical, symbol Connector_Generic:Conn_01x02
- removed J508: PWR OUT2, Connector_Phoenix_MC:PhoenixContact_MCV_1,5_2-G-3.5_1x02_P3.50mm_Vertical, symbol Connector_Generic:Conn_01x02
- added J501: OUT1, Connector_Phoenix_MC:PhoenixContact_MCV_1,5_4-G-3.5_1x04_P3.50mm_Vertical, symbol Connector_Generic:Conn_02x02_Top_Bottom
- added J502: OUT2, Connector_Phoenix_MC:PhoenixContact_MCV_1,5_4-G-3.5_1x04_P3.50mm_Vertical, symbol Connector_Generic:Conn_02x02_Top_Bottom
- added J503: PWR, Connector_Phoenix_MC:PhoenixContact_MCV_1,5_4-G-3.5_1x04_P3.50mm_Vertical, symbol Connector_Generic:Conn_02x02_Top_Bottom
- added J505: PWR_IN, Connector_PinHeader_2.54mm:PinHeader_2x02_P2.54mm_Vertical, symbol Connector_Generic:Conn_01x04
Connections:
- net +VSW: now also J501.1 (Pin_1), J501.3 (Pin_3), J502.1 (Pin_1), J502.3 (Pin_3), J503.1 (Pin_1), J503.3 (Pin_3), J505.1 (Pin_1), J505.2 (Pin_2)
- net GND: now also J503.2 (Pin_2), J503.4 (Pin_4), J505.3 (Pin_3), J505.4 (Pin_4)
- net at D504.1 (K), Q504.5 (D), Q504.6 (D)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: now also J502.4 (Pin_4)
- net at D503.1 (K), Q503.5 (D), Q503.6 (D)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: now also J502.2 (Pin_2)
- net at D502.1 (K), Q502.5 (D), Q502.6 (D)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: now also J501.4 (Pin_4)
- net at D501.1 (K), Q501.5 (D), Q501.6 (D)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: now also J501.2 (Pin_2)
