File: electronics/RovHat/power.kicad_sch (KiCad schematic)
At the start: 17 parts, among them J501 OUT1, J502 OUT2, J503 PWR, J504 5V IN, J505 PWR_IN, Q501 IRF7403, Q502 IRF7403, Q503 IRF7403, Q504 IRF7403

Commit message: Multiple fixes
Parts:
- removed D501, D502: MBR0550, Diode_SMD:D_SOD-123, symbol Diode:MBR0550
- removed J501: OUT1, Connector_Phoenix_MC:PhoenixContact_MCV_1,5_4-G-3.5_1x04_P3.50mm_Vertical, symbol Connector_Generic:Conn_02x02_Top_Bottom
- removed Q501, Q502: IRF7403, Package_SO:SOIC-8_3.9x4.9mm_P1.27mm, symbol Transistor_FET:IRF7403
- removed R501, R502: R_Small, Resistor_SMD:R_0603_1608Metric, symbol Device:R_Small
- added F1, F2, F3: Polyfuse, Fuse:Fuse_1206_3216Metric, symbol Device:Polyfuse
- J15: renamed from J505; value PWR_IN -> PWR_STACK
- R17: renamed from R503; value R_Small -> 10k; symbol Device:R_Small -> Resistors_0603:RESC_0603_10k; Package (none) -> 0603
- R18: renamed from R504; value R_Small -> 10k; symbol Device:R_Small -> Resistors_0603:RESC_0603_10k; Package (none) -> 0603
- renumbered D503 to D1, D504 to D2, J504 to J12, J503 to J13, J502 to J14, Q503 to Q1, Q504 to Q2
Connections:
- net CH3 is gone; now on net CH1: Q1.4 (G), R17.1
- net CH4 is gone; now on net CH2: Q2.4 (G), R18.1
- net +VSW: now also F1.1, F2.2, F3.1; no longer J13.3 (Pin_3), J14.1 (Pin_1), J14.3 (Pin_3)
- net CH2 OUT: now reaches D2.1 (K), J14.4 (Pin_4), Q2.5 (D), Q2.6 (D), Q2.7 (D), Q2.8 (D)
- net CH1 OUT: now reaches D1.1 (K), J14.2 (Pin_2), Q1.5 (D), Q1.6 (D), Q1.7 (D), Q1.8 (D)
- new net: F2.1, J13.3 (Pin_3)
- new net CH1 FUSED: F1.2, J14.1 (Pin_1)
- new net CH2 FUSED: F3.2, J14.3 (Pin_3)
Other:
- moved on the sheet: D1, D2, J12, J13, J14, J15, Q1, Q2, R17, R18
