File: electronics/RovHat/Connectors.kicad_sch (KiCad schematic)
At the start: 6 parts, among them J401 RPI Header, J402 USB_A, J403 DEPTH, J404 PROPULSION

Commit message: Multiple fixes
Parts:
- removed J402: USB_A, Connector_USB:USB_A_Molex_67643_Horizontal, symbol Connector:USB_A
- removed J404: PROPULSION, Connector_PinHeader_2.54mm:PinHeader_1x06_P2.54mm_Vertical, symbol Connector_Generic:Conn_01x06
- added C2, C3: 2u2, Capacitor_SMD:C_0805_2012Metric, symbol Capacitors_0805:CAPC_2.2uF_X7R_100V_0805
- added J11: Depth, Connector_PinHeader_2.54mm:PinHeader_2x03_P2.54mm_Vertical, symbol Connector_Generic:Conn_02x03_Odd_Even
- added J7: Conn_01x02, Connector_PinHeader_2.54mm:PinHeader_2x01_P2.54mm_Vertical, symbol Connector_Generic:Conn_01x02
- added J8: Servo, Connector_PinHeader_2.54mm:PinHeader_2x03_P2.54mm_Vertical, symbol Connector_Generic:Conn_02x03_Odd_Even
- added JP3: Servo Voltage, Findersee_parts:0402_Jumper_3pin, symbol Jumper:SolderJumper_3_Open
- added R13, R14: 0R, Resistor_SMD:R_0603_1608Metric, symbol Device:R
- J9: renamed from J403; value DEPTH -> Conn_01x08; footprint Connector_PinHeader_2.54mm:PinHeader_1x06_P2.54mm_Vertical -> Connector_JST:JST_SH_SM08B-SRSS-TB_1x08-1MP_P1.00mm_Horizontal; symbol Connector_Generic:Conn_01x06 -> Connector_Generic:Conn_01x08
- renumbered J401 to J10, R401 to R15, R402 to R16
Connections:
- net +5V: now also JP3.1 (A); no longer J9.2 (Pin_2), J9.5 (Pin_5)
- net GND: now also J9.2 (Pin_2), C2.2, C3.2, J11.5 (Pin_5), J11.6 (Pin_6), J7.2 (Pin_2), J8.5 (Pin_5), J8.6 (Pin_6); no longer J9.3 (Pin_3), J9.6 (Pin_6)
- net RPI_I2C_SDA: now reaches J10.3 (Pin_3)
- net RPI_I2C_SCL: now reaches J10.5 (Pin_5)
- net DL: no longer names the net of J9.1 (Pin_1)
- net DL: now also R14.1
- net DR: no longer names the net of J9.4 (Pin_4)
- net DR: now also R13.1
- new net: C2.1, C3.1, J8.3 (Pin_3), J8.4 (Pin_4), JP3.2 (C)
- new net: J7.1 (Pin_1), JP3.3 (B)
- new net CURRENT: R13.2
- new net DEPTH LEFT: J11.1 (Pin_1)
- new net DEPTH RIGHT: J11.2 (Pin_2)
- new net FRONT LEFT: J9.7 (Pin_7)
- new net FRONT RIGHT: J9.8 (Pin_8)
- new net MOT VOLT: R14.2
- new net REAR LEFT: J9.5 (Pin_5)
- new net REAR RIGHT: J9.6 (Pin_6)
- new net Servo 1: J8.1 (Pin_1)
- new net Servo 2: J8.2 (Pin_2)
