File: electronics/RovHat/MCU.kicad_sch (KiCad schematic)
At the start: 4 parts, among them J301 PWM_OUT, J305 SWD_EXT, U301 Rpi_Pico

Commit message: Multiple fixes
Parts:
- J6: renamed from J305; footprint Connector_PinHeader_2.54mm:PinHeader_1x03_P2.54mm_Vertical -> Connector_JST:JST_SH_BM03B-SRSS-TB_1x03-1MP_P1.00mm_Vertical
- R12: renamed from R303; symbol Device:R -> Resistors_0603:RESC_0603_10k; Package (none) -> 0603
- renumbered J301 to J5, U301 to U2
Connections:
- net PWM_3 is gone; now on net PWM_1: U2.22 (GP17)
- net PWM_4 is gone; now on net PWM_2: U2.21 (GP16)
- net ADS_RDY: now also U2.6 (GP4); no longer U2.27 (GP21)
- net GND: no longer U2.43 (TP1(GND))
- net PWM_1: no longer U2.25 (GP19)
- net PWM_2: no longer U2.24 (GP18)
- net at J5.3 (Pin_3): now also U2.4 (GP2); no longer U2.10 (GP7)
- net DEPTH LEFT: now reaches U2.26 (GP20)
- net at U2.5 (GP3): now also J5.2 (Pin_2)
- net RPI_I2C_SDA: now reaches U2.9 (GP6)
- net RPI_I2C_SDA: no longer J5.2 (Pin_2)
- net PIO1 renamed FRONT RIGHT
- net PIO2 renamed FRONT LEFT
- net PIO3 renamed REAR RIGHT
- net PIO4 renamed REAR LEFT
- net USB_D+: no longer names the net of U2.41 (TP3(DP))
- net USB_D-: no longer names the net of U2.42 (TP2(DM))
- new net DEPTH RIGHT: U2.27 (GP21)
- new net RPI_I2C_SCL: U2.10 (GP7)
- new net Servo 1: U2.24 (GP18)
- new net Servo 2: U2.25 (GP19)
- no-connect marks 8 -> 6
Other:
- moved on the sheet: J5
