File: electronics/RovHat/Sensors.kicad_sch (KiCad schematic)
At the start: 15 parts, among them J201 ADS1115, J202 ANALOG INPUT, J203 GYRO, J204 I2C EXPAND

Commit message: Multiple fixes
Parts:
- removed J201: ADS1115, Connector_PinHeader_2.54mm:PinHeader_1x10_P2.54mm_Vertical, symbol Connector_Generic:Conn_01x10
- added C1: 1uf, Capacitor_SMD:C_0603_1608Metric, symbol Capacitors_0603:CAPC_1uf_X5R_10V_0603
- added J3: Conn_01x04, Connector_Molex:Molex_PicoBlade_53398-0471_1x04-1MP_P1.25mm_Vertical, symbol Connector_Generic:Conn_01x04
- added U1: ADS1115IDGS, Package_SO:TSSOP-10_3x3mm_P0.5mm, symbol Analog_ADC:ADS1115IDGS
- R1: renamed from R210; value 4k7 -> 2k2; symbol Device:R_Small -> Resistors_0603_E24:RESC_0603_2k2; Package (none) -> 0603
- R10: renamed from R204; symbol Device:R_Small -> Resistors_0603_E24:RESC_0603_20k; Package (none) -> 0603
- R11: renamed from R209; value 4k7 -> 2k2; symbol Device:R_Small -> Resistors_0603_E24:RESC_0603_2k2; Package (none) -> 0603
- R2: renamed from R211; value 4k7 -> 2k2; symbol Device:R_Small -> Resistors_0603_E24:RESC_0603_2k2; Package (none) -> 0603
- R3: renamed from R205; symbol Device:R_Small -> Resistors_0603:RESC_0603_10k; Package (none) -> 0603
- R4: renamed from R206; symbol Device:R_Small -> Resistors_0603:RESC_0603_10k; Package (none) -> 0603
- R5: renamed from R207; symbol Device:R_Small -> Resistors_0603:RESC_0603_10k; Package (none) -> 0603
- R6: renamed from R208; value 10k -> 180k; symbol Device:R_Small -> Resistors_0603_E24:RESC_0603_180k; Package (none) -> 0603
- R7: renamed from R201; symbol Device:R_Small -> Resistors_0603_E24:RESC_0603_20k; Package (none) -> 0603
- R8: renamed from R202; symbol Device:R_Small -> Resistors_0603_E24:RESC_0603_20k; Package (none) -> 0603
- R9: renamed from R203; symbol Device:R_Small -> Resistors_0603_E24:RESC_0603_20k; Package (none) -> 0603
- renumbered J202 to J1, J203 to J2, J204 to J4
Connections:
- net +5V: now also J3.1 (Pin_1)
- net A0: now also U1.5 (AIN1)
- net A1: now also U1.4 (AIN0)
- net A2: now also U1.7 (AIN3)
- net A3: now also U1.6 (AIN2)
- net ADS_RDY: now also U1.2 (ALERT/RDY)
- net GND: now also C1.1, J3.4 (Pin_4), U1.3 (GND)
- net SCL: now also J3.3 (Pin_3), U1.10 (SCL)
- net SDA: now also J3.2 (Pin_2), U1.9 (SDA)
- net VDD: now also R11.1, C1.2, U1.8 (VDD); no longer R11.2
- net Current: now reaches J1.1 (Pin_1), R3.2
- net MOT VOLT: now reaches J1.7 (Pin_7), R6.2
- new net: R11.2, U1.1 (ADDR)
Other:
- moved on the sheet: J4, R11
