File: electronics/PowerBoard/Leak.kicad_sch (KiCad schematic)
At the start: 21 parts, among them J301 Conn_01x02, J302 Conn_01x02, J303 Conn_01x02, J304 Conn_01x02, U301 LM339

Commit message: Multiple fixes
Parts:
- renumbered C302 to C11, C301 to C12, J301 to J1, J302 to J2, J303 to J3, J304 to J4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
