File: electronics/PowerBoard/SMPS.kicad_sch (KiCad schematic)
At the start: 12 parts, among them U201 XL1509-5.0E1

Commit message: Multiple fixes
Parts:
- removed D201: B340-13F, Diode_SMD:D_SMB, symbol Diode:B340
- removed U201: XL1509-5.0E1, Package_SO:SOIC-8_3.9x4.9mm_P1.27mm, symbol Findersee_parts:XL1509-5.0E1
- added C4, C5: 100nF, Capacitor_SMD:C_0603_1608Metric, symbol Capacitors_0603:CAPC_100nF_X7R_50V_0603
- added D1: B360, Diode_SMD:D_SMC, symbol Diode:B360
- added R1: 4k7, Resistor_SMD:R_0603_1608Metric, symbol Resistors_0603_E24:RESC_0603_4k7
- added R2: 1k5, Resistor_SMD:R_0603_1608Metric, symbol Resistors_0603_E24:RESC_0603_1k5
- added U1: ST1S14PHR, Package_SO:TI_SO-PowerPAD-8, symbol Regulator_Switching:ST1S14PHR
- C2: renamed from C201; value 470uF / 35V -> 330uF / 63V
- C3: renamed from C207; value 1u -> 10u
- L2: renamed from L201; value YSPI1050-680M -> DJNR8040-4R7; footprint Findersee_parts:YSPI1050 -> Inductors SMD:IND_BOURNS_SRN8040; Value 2 68uH / 3A -> 4u7 / 4.5A
- renumbered C202 to C1, C208 to C10, C203 to C6, C204 to C7, C205 to C8, C206 to C9, L202 to L1
Connections:
- net GND: now also C4.2, D1.2 (A), R2.1, U1.3 (~{EN1}), U1.6 (GND), U1.9 (PADGND)
- net VCC: now also R1.1
- net VIN FILT: now also C4.1, U1.5 (EN2), U1.7 (VIN)
- net sw: now also C5.2, D1.1 (K), U1.8 (SW)
- new net: C5.1, U1.1 (BOOT)
- new net: R1.2, R2.2, U1.4 (FB)
Other:
- moved on the sheet: C10, C2, C3, C6, C7, C8, C9, L2
