File: electronics/PowerBoard/PowerBoard.kicad_pcb (KiCad board)
At the start: 2 copper layers, 65 x 56 mm, 42 parts, among them J301 Conn_01x02, J302 Conn_01x02, J303 Conn_01x02, J304 Conn_01x02, J401 Conn_02x20_Odd_Even, J402 PWR Stack, J404 PWR Stack, J405 Conn_01x04, U201 XL1509-5.0E1, U301 LM339

Commit message: PowerBoard commit
Parts:
- removed REF**: ESD-Logo_13.2x12mm_SilkScreen, Symbol:ESD-Logo_13.2x12mm_SilkScreen
- removed REF**: KiCad-Logo2_6mm_SilkScreen, Symbol:KiCad-Logo2_6mm_SilkScreen
- added C401: 1u, Capacitor_SMD:C_0805_2012Metric, F.Cu at (124.0, 103.2)
- added J403: Conn_01x04, Connector_PinSocket_2.54mm:PinSocket_1x04_P2.54mm_Vertical, F.Cu at (192.5, 113.3)
- added J406: PWR Stack, Connector_Phoenix_MC:PhoenixContact_MCV_1,5_4-G-3.5_1x04_P3.50mm_Vertical, F.Cu at (107.0, 51.5)
- added R401: 0R, Resistor_SMD:R_0402_1005Metric, F.Cu at (118.0, 56.5)
- added R402: 0R, Resistor_SMD:R_0402_1005Metric, F.Cu at (118.0, 58.5)
- added R403: 0R, Resistor_SMD:R_0402_1005Metric, F.Cu at (118.0, 60.5)
- added R404: 0R, Resistor_SMD:R_0402_1005Metric, F.Cu at (118.0, 62.5)
- added R405: 4k7, Resistor_SMD:R_0603_1608Metric, F.Cu at (110.1, 63.2)
- added R406: 4k7, Resistor_SMD:R_0603_1608Metric, F.Cu at (110.1, 65.8)
- added U401: ~, Package_SO:SOIC-8_3.9x4.9mm_P1.27mm, F.Cu at (185.3, 126.4)

Commit message: Multiple fixes
Parts:
- removed C401: 1u, Capacitor_SMD:C_0805_2012Metric
- removed D201: B340-13F, Diode_SMD:D_SMB
- removed J405: Conn_01x04, Connector_PinSocket_2.54mm:PinSocket_1x04_P2.54mm_Vertical
- removed J406: PWR Stack, Connector_Phoenix_MC:PhoenixContact_MCV_1,5_4-G-3.5_1x04_P3.50mm_Vertical
- removed R401, R402, R403, R404: 0R, Resistor_SMD:R_0402_1005Metric
- removed U201: XL1509-5.0E1, Package_SO:SOIC-8_3.9x4.9mm_P1.27mm
- removed U401: ~, Package_SO:SOIC-8_3.9x4.9mm_P1.27mm
- added C4: 100nF, Capacitor_SMD:C_0603_1608Metric, F.Cu at (128.8, 108.2)
- added C5: 100nF, Capacitor_SMD:C_0603_1608Metric, F.Cu at (129.3, 101.0)
- added D1: B360, Diode_SMD:D_SMC, F.Cu at (139.1, 106.9)
- added H4: MountingHole, MountingHole:MountingHole_2.7mm_M2.5, F.Cu at (168.5, 133.5)
- added J7: I2C Pressure, Connector_Molex:Molex_PicoBlade_53398-0471_1x04-1MP_P1.25mm_Vertical, F.Cu at (169.3, 123.2)
- added R1: 4k7, Resistor_SMD:R_0603_1608Metric, F.Cu at (129.6, 99.0)
- added R2: 1k5, Resistor_SMD:R_0603_1608Metric, F.Cu at (122.3, 107.3)
- added U1: ST1S14PHR, Package_SO:TI_SO-PowerPAD-8, F.Cu at (127.3, 104.6)
- C2: renamed from C201; value 470uF / 35V -> 330uF / 63V
- C3: renamed from C207; value 1u -> 10u
- J6: renamed from J403; value Conn_01x04 -> I2C2
- J9: renamed from J402; value PWR Stack -> PWR IN
- L2: renamed from L201; value YSPI1050-680M -> DJNR8040-4R7; footprint Findersee_parts:YSPI1050 -> Inductors SMD:IND_BOURNS_SRN8040
- moved J6 76.7 mm to (117.8, 95.7), turned to 90 degrees
- moved R17 30.0 mm to (119.5, 91.7)
- moved R18 29.1 mm to (119.5, 93.2)
- moved C10 10.8 mm to (142.0, 96.8), turned to 0 degrees
- moved C8 9.83 mm to (142.0, 94.5), turned to 0 degrees
- moved C6 5.12 mm to (129.5, 94.8)
- moved C7 5.12 mm to (129.5, 92.5)
- moved C9 5.12 mm to (129.5, 97.0)
- moved C12 4.67 mm to (152.4, 115.6)
- moved R3 4.28 mm to (157.7, 113.8), turned to -90 degrees
- moved R4 4.07 mm to (152.6, 113.7), turned to 180 degrees
- moved L2 3.89 mm to (135.6, 99.3)
- moved C2 1.24 mm to (128.7, 117.2)
- moved C3 0.96 mm to (128.8, 110.2)
- renumbered C202 to C1, C208 to C10, C302 to C11, C301 to C12, C203 to C6, C204 to C7, C205 to C8, C206 to C9, H401 to H1, H402 to H2, H403 to H3, J301 to J1, J302 to J2, J303 to J3, J304 to J4, J401 to J5, J404 to J8, L202 to L1, R306 to R10, R307 to R11, R313 to R12, R308 to R13, R314 to R14, R309 to R15, R310 to R16, R405 to R17, R406 to R18, R301 to R3, R302 to R4, R303 to R5, R311 to R6, R304 to R7, R312 to R8, R305 to R9, U301 to U2
Routing:
- net /Connectors/SDA: track 22.1 -> 100.2 mm, vias 0 -> 2
- net /Connectors/SCL: track 11.7 -> 88.3 mm, vias 0 -> 2
- net Net-(U1-FB): track 0.00 -> 14.5 mm
- net VDD: track 25.7 -> 33.4 mm
- net /SMPS/VIN FILT: track 0.00 -> 6.54 mm
- net VCC: track 80.6 -> 87.0 mm
- net Net-(U1-BOOT): track 0.00 -> 5.40 mm
- net +2V5: track 35.0 -> 36.5 mm
- net GND: vias 66 -> 74
Other:
- outline, holes or cut-outs redrawn
- board text added: "+ -"
- board text added: "Findersee 23/26"
- board text removed: "+ - + -"
- board text removed: "Findersee 03/23"
