File: electronics/Power_Drum/Power_Drum.kicad_pcb (KiCad board)
At the start: 2 copper layers, 85 x 45 mm, 46 parts, among them J1 BAT 1, J2 DC IN, J3 BAT 2, J4 OUTPUT, J5 PowerLine, J6 WiFi, J7 LED, Q1 2N7002, Q2 BSC098N10NS5, Q3 BSC098N10NS5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

Commit message: Power Drum V2 update
Parts:
- removed C2: 100nF, Capacitor_SMD:C_0603_1608Metric
- removed C5: 470uF, Capacitor_THT:CP_Radial_D10.0mm_P5.00mm
- removed D1, D2: SK2040YD2R, Package_TO_SOT_SMD:TO-263-2
- removed R2: 47k, Resistor_SMD:R_0603_1608Metric
- removed R3: 120k, Resistor_SMD:R_0603_1608Metric
- removed R4, R7: 3k3, Resistor_SMD:R_0603_1608Metric
- removed R9: 0R, Resistor_SMD:R_0402_1005Metric
- removed the U1 at (145.2, 105.0)
- added C15: 100nF, Capacitor_SMD:C_0603_1608Metric, F.Cu at (152.8, 120.1)
- added C16: 2u2, Capacitor_SMD:C_0805_2012Metric, F.Cu at (141.6, 120.6)
- added C17: 2u2, Capacitor_SMD:C_0805_2012Metric, F.Cu at (139.0, 104.7)
- added C18: 100nF, Capacitor_SMD:C_0603_1608Metric, F.Cu at (149.5, 125.8)
- added J10: TRIP LED, Connector_PinHeader_2.54mm:PinHeader_1x02_P2.54mm_Vertical, F.Cu at (156.4, 130.2)
- added J8: COMMS, Connector_PinHeader_2.54mm:PinHeader_1x02_P2.54mm_Vertical, F.Cu at (174.7, 122.7)
- added J9: RESET SW, Connector_PinHeader_2.54mm:PinHeader_1x02_P2.54mm_Vertical, F.Cu at (189.8, 124.0)
- added JP1: 5V Regulator Select, Connector_PinHeader_2.54mm:PinHeader_1x03_P2.54mm_Vertical, F.Cu at (163.9, 107.4)
- added Q4: BSC098N10NS5, Package_TO_SOT_SMD:TDSON-8-1, F.Cu at (154.8, 115.2)
- added R12: 120k, Resistor_SMD:R_0603_1608Metric, F.Cu at (144.3, 123.5)
- added R13: 3k3, Resistor_SMD:R_0603_1608Metric, F.Cu at (144.5, 127.0)
- added R14: 91k, Resistor_SMD:R_0603_1608Metric, F.Cu at (154.2, 120.1)
- added R15: 3k3, Resistor_SMD:R_0603_1608Metric, F.Cu at (146.5, 124.8)
- added R16: 0R, Resistor_SMD:R_0603_1608Metric, F.Cu at (149.5, 124.0)
- added R17: 3k3, Resistor_SMD:R_0603_1608Metric, F.Cu at (193.1, 124.0)
- added R18: 3k3, Resistor_SMD:R_0603_1608Metric, F.Cu at (178.6, 132.0)
- added R19: 3k3, Resistor_SMD:R_0603_1608Metric, F.Cu at (187.1, 130.6)
- added R20: 3k3, Resistor_SMD:R_0603_1608Metric, F.Cu at (187.1, 127.4)
- added R21: 120k, Resistor_SMD:R_0603_1608Metric, F.Cu at (172.2, 129.4)
- added TP1: Current, TestPoint:TestPoint_Pad_D1.5mm, F.Cu at (189.2, 129.7)
- added TP2: TestPoint, TestPoint:TestPoint_Pad_D1.5mm, F.Cu at (191.8, 132.9)
- added U2: INA202DGK, Package_SO:VSSOP-8_3x3mm_P0.65mm, F.Cu at (184.3, 126.1)
- added U4: LM74801QDRRRQ1, Package_SON:WSON-12-1EP_3x3mm_P0.5mm_EP1.5x2.5mm, F.Cu at (147.9, 120.0)
- C10: footprint Capacitor_THT:CP_Radial_D10.0mm_P5.00mm -> Capacitor_THT:CP_Radial_D12.5mm_P5.00mm
- C9: value 470uF -> 100nF; footprint Capacitor_THT:CP_Radial_D10.0mm_P5.00mm -> Capacitor_SMD:C_0603_1608Metric
- L1: value DJNR8040-100 -> DJNR8040-6R8
- Q1: value 2N7002 -> BC817
- R1: value 120k -> ~0.971mohm; footprint Resistor_SMD:R_0603_1608Metric -> Findersee_parts:SHUNT_5x8
- R10: value 9k1 -> 4k7
- R11: value 1k0 -> 1k5
- moved C9 33.9 mm to (182.5, 130.2), turned to 0 degrees
- moved R1 24.9 mm to (183.6, 118.0), turned to 0 degrees
- moved U1 23.7 mm to (145.2, 105.0)
- moved C3 23.4 mm to (142.6, 105.0)
- moved Q3 22.7 mm to (147.3, 100.0)
- moved R6 22.3 mm to (146.5, 109.5), turned to 180 degrees
- moved C1 21.9 mm to (141.0, 105.0), turned to -90 degrees
- moved R8 21.7 mm to (146.5, 111.1), turned to 180 degrees
- moved R5 19.0 mm to (147.7, 107.0)
- moved C4 16.0 mm to (143.6, 120.4), turned to -90 degrees
- moved Q2 15.3 mm to (146.6, 115.2)
- moved C7 9.67 mm to (174.7, 118.2), turned to 90 degrees
- moved J2 6.14 mm to (128.6, 101.0)
- moved Q1 3.76 mm to (168.2, 131.2)
- moved C10 3.73 mm to (164.5, 119.3)
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- renumbered U2 to U1
Connections:
- net Net-(D1-K) renamed /Batt Centre
- C1 pad 1: +BATT -> VDC
- C12 pad 1: +12V -> +5V
- C13 pad 1: +12V -> +5V
- C14 pad 1: +12V -> +5V
- C3 pad 1: +BATT -> VDC
- C4 pad 1: VDC -> +BATT
- C6 pad 1: +36V -> Net-(JP1-C)
- C8 pad 1: +36V -> Net-(JP1-C)
- C9 pad 1: +36V -> GND
- C9 pad 2: GND -> +5V
- J4 pad 1: +36V -> /VOUT
- J5 pad 1: +12V -> +5V
- J6 pad 1: +12V -> +5V
- J7 pad 1: +12V -> +5V
- L1 pad 2: +12V -> +5V
- Q1 pad 1: /BATTERY DISABLE -> Net-(Q1-B)
- Q2 pad 1: VDC -> +BATT
- Q2 pad 2: VDC -> +BATT
- Q2 pad 3: VDC -> +BATT
- Q2 pad 4: Net-(Q2-G) -> /Dgate
- Q2 pad 5: +36V -> /Cathode
- Q3 pad 1: +BATT -> VDC
- Q3 pad 2: +BATT -> VDC
- Q3 pad 3: +BATT -> VDC
- Q3 pad 5: +36V -> /Cathode
- R1 pad 1: VDC -> +36V
- R1 pad 2: /BATTERY DISABLE -> Net-(U2-V_{IN+})
- R10 pad 1: +12V -> +5V
- R5 pad 1: +BATT -> VDC
- U1 pad 4: +36V -> /Cathode
- U1 pad 6: +BATT -> VDC
- U3 pad 5: +36V -> Net-(JP1-C)
- U3 pad 7: +36V -> Net-(JP1-C)
Routing:
- net +5V: track 0.00 -> 89.7 mm
- net Net-(U2-CMP_{OUT}): track 0.00 -> 55.7 mm
- net +12V: track 33.0 -> 0.00 mm
- net VDC: track 35.4 -> 5.26 mm
- net /Hgate: track 0.00 -> 18.6 mm, vias 0 -> 2
- net /Cathode: track 0.00 -> 17.2 mm, vias 0 -> 2
- net Net-(J10-Pin_1): track 5.83 -> 22.1 mm
- net Net-(U2-OUT): track 0.00 -> 8.99 mm
- net /BATTERY DISABLE: track 7.29 -> 0.00 mm
- net Net-(U2-V_{IN+}): track 0.00 -> 7.26 mm
- net Net-(U2-V_{IN-}): track 0.00 -> 7.20 mm
- net Net-(U1-EN): track 13.6 -> 6.50 mm
- net Net-(J9-Pin_1): track 0.00 -> 7.01 mm
- net Net-(U4-OV): track 0.00 -> 6.88 mm
- net Net-(JP1-C): track 0.00 -> 6.07 mm
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- added copper zone on F.Cu, net +5V
- added copper zone on F.Cu, net /Cathode
- added copper zone on F.Cu, net /VOUT
- added copper zone on F.Cu, net Net-(JP1-C)
- removed copper zone on F.Cu, net +12V
- removed copper zone on F.Cu, net +BATT
- removed copper zone on F.Cu, net /Batt Centre
Other:
- rule pad_to_mask_clearance: 0 -> 0.02
- board text added: "+"
- board text added: "-"

Commit message: Manufacturing commit
Parts:
- removed R20: 3k3, Resistor_SMD:R_0603_1608Metric
- added C19: 100nF, Capacitor_SMD:C_0603_1608Metric, F.Cu at (154.2, 95.5)
- added C2: 220nF, Capacitor_SMD:C_0402_1005Metric, F.Cu at (183.4, 120.2)
- added J11: Conn_01x03, Connector_PinHeader_2.54mm:PinHeader_1x03_P2.54mm_Vertical, F.Cu at (151.0, 132.4)
- added J12: Current Out, Connector_PinHeader_2.54mm:PinHeader_1x02_P2.54mm_Vertical, F.Cu at (182.1, 130.1)
- added J13: 5V Spare, Connector_PinHeader_2.54mm:PinHeader_1x02_P2.54mm_Vertical, F.Cu at (193.7, 101.6)
- added Q5: BC817, Package_TO_SOT_SMD:SOT-23, F.Cu at (173.1, 129.2)
- added R2: 100R, Resistor_SMD:R_0402_1005Metric, F.Cu at (179.8, 122.3)
- added R3: 100R, Resistor_SMD:R_0402_1005Metric, F.Cu at (186.6, 121.7)
- added REF**: KiCad-Logo2_8mm_SilkScreen, Symbol:KiCad-Logo2_8mm_SilkScreen, B.Cu at (127.0, 112.9)
- added RV1: 5k, Potentiometer_SMD:Potentiometer_Bourns_3314G_Vertical, F.Cu at (188.4, 130.6)
- J10, J7, J9: footprint Connector_PinHeader_2.54mm:PinHeader_1x02_P2.54mm_Vertical -> Connector_Molex:Molex_KK-254_AE-6410-02A_1x02_P2.54mm_Vertical
- R18, R19: value 3k3 -> 150R
- R21: value 120k -> 1k5
- TP1: value Current -> Setpoint; footprint TestPoint:TestPoint_Pad_D1.5mm -> TestPoint:TestPoint_Pad_D1.0mm
- TP2: value TestPoint -> GND; footprint TestPoint:TestPoint_Pad_D1.5mm -> TestPoint:TestPoint_Pad_D1.0mm
- moved R19 24.8 mm to (190.3, 106.0), turned to -90 degrees
- moved R18 17.5 mm to (161.2, 132.1), turned to 90 degrees
- moved R21 10.2 mm to (181.1, 124.4)
- moved TP2 9.62 mm to (198.3, 125.9)
- moved J7 7.22 mm to (185.7, 107.3), turned to -90 degrees
- moved C9 5.96 mm to (186.3, 125.6), turned to 90 degrees
- moved TP1 5.36 mm to (193.1, 133.3)
- moved JP1 5.08 mm to (158.9, 107.4), turned to 90 degrees
- moved R17 3.76 mm to (196.4, 122.2)
- moved U2 2.26 mm to (183.6, 124.0)
- moved J9 2.01 mm to (191.2, 125.4), turned to 90 degrees
- moved R11 1.65 mm to (156.2, 101.5), turned to -90 degrees
- moved Q1 0.87 mm to (169.1, 131.3), turned to 90 degrees
- moved J10 0.79 mm to (156.5, 130.9), turned to 90 degrees
Connections:
- J10 pad 2: GND -> Net-(J10-Pin_2)
- J7 pad 1: +5V -> Net-(J7-Pin_1)
- JP1 pad 1: +36V -> /Cathode
- JP1 pad 3: /Cathode -> +36V
- Q1 pad 3: Net-(J10-Pin_1) -> Net-(J10-Pin_2)
- R1 pad 2: Net-(U2-V_{IN+}) -> Net-(R1-Pad2)
- R1 pad 3: Net-(U2-V_{IN-}) -> Net-(R1-Pad3)
- R14 pad 2: Net-(U2-CMP_{OUT}) -> Net-(Q5-C)
- R15 pad 1: Net-(U2-CMP_{OUT}) -> Net-(Q5-C)
- R19 pad 1: Net-(U2-OUT) -> +5V
- R19 pad 2: Net-(U2-CMP_{IN}) -> Net-(J7-Pin_1)
- R21 pad 1: Net-(Q1-B) -> +5V
- R21 pad 2: Net-(U2-CMP_{OUT}) -> Net-(Q1-B)
- TP1 pad 1: Net-(U2-OUT) -> Net-(U2-CMP_{IN})
- U2 pad 2: Net-(U2-OUT) -> Net-(J12-Pin_1)
- U2 pad 6: Net-(U2-CMP_{OUT}) -> Net-(Q1-B)
- U4 pad 6: Net-(U2-CMP_{OUT}) -> Net-(Q5-C)
Routing:
- net Net-(U2-CMP_{OUT}): track 55.7 -> 0.00 mm
- net Net-(Q5-C): track 0.00 -> 41.8 mm
- net +5V: track 89.7 -> 113.9 mm
- net Net-(Q1-B): track 4.94 -> 25.3 mm
- net Net-(J10-Pin_1): track 22.1 -> 4.79 mm
- net Net-(J11-Pin_2): track 3.87 -> 18.7 mm
- net Net-(J10-Pin_2): track 0.00 -> 13.7 mm
- net Net-(J12-Pin_1): track 0.00 -> 9.03 mm
- net Net-(U2-OUT): track 8.99 -> 0.00 mm
- net Net-(U2-CMP_{IN}): track 5.36 -> 13.8 mm
- net Net-(J9-Pin_1): track 7.01 -> 15.4 mm
- net Net-(J7-Pin_1): track 0.00 -> 4.83 mm
- net Net-(U2-V_{IN-}): track 7.20 -> 5.18 mm
- net Net-(R1-Pad2): track 0.00 -> 1.98 mm
- net Net-(R1-Pad3): track 0.00 -> 1.97 mm
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Other:
- outline, holes or cut-outs redrawn
- board text added: "${REVISION}|${CURRENT_DATE}"
- board text added: "- + - +"
- board text added: "H"
- board text added: "P"
