File: electronics/Power_Drum/Power_Drum.kicad_sch (KiCad schematic)
At the start: 46 parts, among them J1 BAT 1, J2 DC IN, J3 BAT 2, J4 OUTPUT, J5 PowerLine, J6 WiFi, J7 LED, Q1 2N7002, Q2 BSC098N10NS5, Q3 BSC098N10NS5, U1 LM74700, U2 LM74700, U3 ST1S14PHR

Commit message: Power Drum V2 update
Parts:
- removed C2: 100nF, Capacitor_SMD:C_0603_1608Metric, symbol Capacitors_0603:CAPC_100nF_X7R_50V_0603
- removed C5, C9: 470uF, Capacitor_THT:CP_Radial_D10.0mm_P5.00mm, symbol Findersee_parts:CAPEL_470uF_100V
- removed D1, D2: SK2040YD2R, Package_TO_SOT_SMD:TO-263-2, symbol Device:D_Schottky_AKA
- removed Q1: 2N7002, Package_TO_SOT_SMD:SOT-23, symbol Transistor_FET:2N7002
- removed R1, R3: 120k, Resistor_SMD:R_0603_1608Metric, symbol Resistors_0603_E24:RESC_0603_120k
- removed R2: 47k, Resistor_SMD:R_0603_1608Metric, symbol Resistors_0603_E24:RESC_0603_47k
- removed R4, R7: 3k3, Resistor_SMD:R_0603_1608Metric, symbol Resistors_0603_E24:RESC_0603_3k3
- removed R9: 0R, Resistor_SMD:R_0402_1005Metric, symbol Resistors_0402_E24:RESC_0402_0R
- removed U1: LM74700, Package_TO_SOT_SMD:SOT-23-6, symbol Power_Management:LM74700
- added C15, C18, C9: 100nF, Capacitor_SMD:C_0603_1608Metric, symbol Capacitors_0603:CAPC_100nF_X7R_50V_0603
- added C16, C17: 2u2, Capacitor_SMD:C_0805_2012Metric, symbol Capacitors_0805:CAPC_2.2uF_X7R_100V_0805
- added J10: TRIP LED, Connector_PinHeader_2.54mm:PinHeader_1x02_P2.54mm_Vertical, symbol Connector_Generic:Conn_01x02
- added J8: COMMS, Connector_PinHeader_2.54mm:PinHeader_1x02_P2.54mm_Vertical, symbol Connector_Generic:Conn_01x02
- added J9: RESET SW, Connector_PinHeader_2.54mm:PinHeader_1x02_P2.54mm_Vertical, symbol Connector_Generic:Conn_01x02
- added JP1: 5V Regulator Select, Connector_PinHeader_2.54mm:PinHeader_1x03_P2.54mm_Vertical, symbol Jumper:Jumper_3_Bridged12
- added Q1: BC817, Package_TO_SOT_SMD:SOT-23, symbol Transistor_BJT:BC817
- added Q4: BSC098N10NS5, Package_TO_SOT_SMD:TDSON-8-1, symbol Transistor_FET:BSC098N10NS5
- added R1: ~0.971mohm, Findersee_parts:SHUNT_5x8, symbol Device:R_Shunt
- added R12, R21: 120k, Resistor_SMD:R_0603_1608Metric, symbol Resistors_0603_E24:RESC_0603_120k
- added R13, R15, R17, R18, R19, R20: 3k3, Resistor_SMD:R_0603_1608Metric, symbol Resistors_0603_E24:RESC_0603_3k3
- added R14: 91k, Resistor_SMD:R_0603_1608Metric, symbol Resistors_0603_E24:RESC_0603_91k
- added R16: 0R, Resistor_SMD:R_0603_1608Metric, symbol Resistors_0603_E24:RESC_0603_0R
- added TP1: Current, TestPoint:TestPoint_Pad_D1.5mm, symbol Connector:TestPoint
- added TP2: TestPoint, TestPoint:TestPoint_Pad_D1.5mm, symbol Connector:TestPoint
- added U2: INA202DGK, Package_SO:VSSOP-8_3x3mm_P0.65mm, symbol Amplifier_Current:INA202DGK
- added U4: LM74801QDRRRQ1, Package_SON:WSON-12-1EP_3x3mm_P0.5mm_EP1.5x2.5mm, symbol Findersee_parts:LM74801-Q1
- C10: footprint Capacitor_THT:CP_Radial_D10.0mm_P5.00mm -> Capacitor_THT:CP_Radial_D12.5mm_P5.00mm
- R10: value 9k1 -> 4k7; symbol Resistors_0603_E24:RESC_0603_9k1 -> Resistors_0603_E24:RESC_0603_4k7
- R11: value 1k0 -> 1k5; symbol Resistors_0603_E24:RESC_0603_1k0 -> Resistors_0603_E24:RESC_0603_1k5
- renumbered U2 to U1
Connections:
- net +36V: now also J8.1 (Pin_1), JP1.1 (A), Q4.1 (S), Q4.2 (S), Q4.3 (S), R1.1, U4.9 (OUT); no longer C6.1, C8.1, J4.1 (Pin_1), Q2.5 (D), Q3.5 (D), U1.4 (CATHODE), U3.5 (EN2), U3.7 (VIN)
- net +5V: now also C9.2, R17.1, R18.1, U2.1 (V_{s})
- net +BATT: now also C4.1, Q2.1 (S), Q2.2 (S), Q2.3 (S), C16.1, U4.2 (A); no longer C1.1, C3.1, Q3.1 (S), Q3.2 (S), Q3.3 (S), R5.1, U1.6 (ANODE)
- net GND: now also C16.2, C17.2, C18.1, C9.1, J10.2 (Pin_2), J8.2 (Pin_2), J9.2 (Pin_2), Q1.2 (E), R13.2, R15.2, R20.2, TP2.1, U2.4 (GND), U4.7 (GND)
- net VDC: now also C1.1, C3.1, Q3.1 (S), Q3.2 (S), Q3.3 (S), R5.1, U1.6 (ANODE), C17.1; no longer C4.1, Q2.1 (S), Q2.2 (S), Q2.3 (S)
- net Batt Centre: now reaches J1.2 (Pin_2), J3.1 (Pin_1)
- net Dgate: now reaches Q2.4 (G)
- net Dgate: now also U4.1 (DGATE)
- new net: J9.1 (Pin_1), R17.2, U2.5 (~{RESET})
- new net: R19.2, R20.1, U2.3 (CMP_{IN})
- new net: R14.2, R15.1, R21.2, U2.6 (CMP_{OUT}), U4.6 (EN/UVLO)
- new net: Q1.1 (B), R21.1
- new net: C6.1, C8.1, JP1.2 (C), U3.5 (EN2), U3.7 (VIN)
- new net: C18.2, R16.2
- new net: J10.1 (Pin_1), Q1.3 (C), R18.2
- new net: R19.1, TP1.1, U2.2 (OUT)
- new net: C15.1, U4.11 (CAP)
- new net: R12.1, U4.4 (SW)
- new net: R12.2, R13.1, U4.5 (OV)
- new net: R1.3, U2.7 (V_{IN-})
- new net: R1.2, U2.8 (V_{IN+})
- new net Cathode: C15.2, JP1.3 (B), Q2.5 (D), Q3.5 (D), Q4.5 (D), R14.1, U1.4 (CATHODE), U4.10 (VS), U4.12 (C), U4.3 (VSNS)
- new net Hgate: Q4.4 (G), R16.1, U4.8 (HGATE)
- new net VOUT: J4.1 (Pin_1), R1.4
Other:
- note added: "Over Voltage 45.99V [43.79V ... 48.27V]"
- note added: "UVLO 32.35V [30.58V ... 33.76V]"
- title: (none) -> Power Drum
- moved on the sheet: C10, C11, C12, C13, C14, C4, C6, C7, C8, D3, H1, H2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

Commit message: Manufacturing commit
Parts:
- removed R19, R20: 3k3, Resistor_SMD:R_0603_1608Metric, symbol Resistors_0603_E24:RESC_0603_3k3
- removed R21: 120k, Resistor_SMD:R_0603_1608Metric, symbol Resistors_0603_E24:RESC_0603_120k
- added C19: 100nF, Capacitor_SMD:C_0603_1608Metric, symbol Capacitors_0603:CAPC_100nF_X7R_50V_0603
- added C2: 220nF, Capacitor_SMD:C_0402_1005Metric, symbol Capacitors_0402:CAPC_220nF_X5R_10V_0402
- added J11: Conn_01x03, Connector_PinHeader_2.54mm:PinHeader_1x03_P2.54mm_Vertical, symbol Connector_Generic:Conn_01x03
- added J12: Current Out, Connector_PinHeader_2.54mm:PinHeader_1x02_P2.54mm_Vertical, symbol Connector_Generic:Conn_01x02
- added J13: 5V Spare, Connector_PinHeader_2.54mm:PinHeader_1x02_P2.54mm_Vertical, symbol Connector_Generic:Conn_01x02
- added Q5: BC817, Package_TO_SOT_SMD:SOT-23, symbol Transistor_BJT:BC817
- added R19: 150R, Resistor_SMD:R_0603_1608Metric, symbol Resistors_0603_E24:RESC_0603_150R
- added R2, R3: 100R, Resistor_SMD:R_0402_1005Metric, symbol Resistors_0402_E24:RESC_0402_100R
- added R21: 1k5, Resistor_SMD:R_0603_1608Metric, symbol Resistors_0603_E24:RESC_0603_1k5
- added RV1: 5k, Potentiometer_SMD:Potentiometer_Bourns_3314G_Vertical, symbol Device:R_Potentiometer_Trim
- C10, C7: value 470uF -> 330uF
- J10, J7, J9: footprint Connector_PinHeader_2.54mm:PinHeader_1x02_P2.54mm_Vertical -> Connector_Molex:Molex_KK-254_AE-6410-02A_1x02_P2.54mm_Vertical
- J8: now left out of the parts list
- R18: value 3k3 -> 150R; symbol Resistors_0603_E24:RESC_0603_3k3 -> Resistors_0603_E24:RESC_0603_150R
- TP1: value Current -> Setpoint; footprint TestPoint:TestPoint_Pad_D1.5mm -> TestPoint:TestPoint_Pad_D1.0mm
- TP2: value TestPoint -> GND; footprint TestPoint:TestPoint_Pad_D1.5mm -> TestPoint:TestPoint_Pad_D1.0mm
- U4: value LM74801QDRRRQ1 -> LM74800QDRRRQ1; symbol Findersee_parts:LM74801-Q1 -> Findersee_parts:LM74800-Q1; Manufacturer Code LM74801QDRRRQ1 -> LM74800QDRRRQ1
Connections:
- net +36V: now also JP1.3 (B); no longer JP1.1 (A)
- net +5V: now also C19.2, J11.1 (Pin_1), J13.1 (Pin_1), R19.1, R21.1; no longer J7.1 (Pin_1)
- net Cathode: now also JP1.1 (A); no longer JP1.3 (B)
- net GND: now also J11.3 (Pin_3), J12.2 (Pin_2), J13.2 (Pin_2), Q5.2 (E), RV1.3; no longer J10.2 (Pin_2)
- net at U2.3 (CMP_{IN}): now also TP1.1, RV1.2
- net at R14.2, R15.1, U4.6 (EN/UVLO): now also Q5.3 (C); no longer U2.6 (CMP_{OUT})
- net at R10.2, R11.1, U3.4 (FB): now also C19.1
- net at Q1.1 (B): now also U2.6 (CMP_{OUT}), Q5.1 (B), R21.2
- net at J10.1 (Pin_1), R18.2: no longer Q1.3 (C)
- net at U2.2 (OUT): now also J12.1 (Pin_1), RV1.1; no longer TP1.1
- net at R12.1, U4.4 (SW): now also J11.2 (Pin_2)
- net at U2.7 (V_{IN-}): now also C2.2, R3.1; no longer R1.3
- net at U2.8 (V_{IN+}): now also C2.1, R2.1; no longer R1.2
- new net: R1.3, R3.2
- new net: J10.2 (Pin_2), Q1.3 (C)
- new net: R1.2, R2.2
- new net: J7.1 (Pin_1), R19.2
Other:
- moved on the sheet: C12, C13, C14, J10, J5, J6, J7, J9, Q1, R17, R18
